File: kicad/r-map_v2/breakout_board/temperature_humidity/temperature_humidity.sch (KiCad schematic (older format))
At the start: 13 parts, among them IC1 ADT7420, P3 CONN_01X04, P4 A0, U1 HIH6100, U2 HIH6100-SOIC8

Commit message: Aggiornamento files gerber e verifica per nuova stampa pcb, revisionate tutte e 4 le board. Il file kicad/r-map_v2/futura_10-2015.zip contiene i files divisi per cartelle di tutte le board
Parts:
- C1: value C -> 0.22uF
- C2, C3: value C -> 0.1uF
Changed lines of the file:
@@
 P 3400 5600
 F 0 "C2" H 3425 5700 50  0000 L CNN
-F 1 "C" H 3425 5500 50  0000 L CNN
+F 1 "0.1uF" H 3425 5500 50  0000 L CNN
 F 2 "w_smd_cap:c_0805" H 3438 5450 30  0001 C CNN
 F 3 "" H 3400 5600 60  0000 C CNN
@@
 P 3050 5600
 F 0 "C1" H 3075 5700 50  0000 L CNN
-F 1 "C" H 3075 5500 50  0000 L CNN
+F 1 "0.22uF" H 3075 5500 50  0000 L CNN
 F 2 "w_smd_cap:c_0805" H 3088 5450 30  0001 C CNN
 F 3 "" H 3050 5600 60  0000 C CNN
@@
 P 5700 3050
 F 0 "C3" H 5725 3150 50  0000 L CNN
-F 1 "C" H 5725 2950 50  0000 L CNN
+F 1 "0.1uF" H 5725 2950 50  0000 L CNN
 F 2 "w_smd_cap:c_0805" H 5738 2900 30  0001 C CNN
 F 3 "" H 5700 3050 60  0000 C CNN

Commit message: Nuova versione breakout board, inviata a servizio di stampa pcb
Parts:
- added R1, R2: R, w_smd_resistors:r_0805, symbol R
Connections:
- net +3V3: now also R1.1, R2.1
- net SCL: now also R2.2
- net SDA: now also R1.2
Other:
- moved on the sheet: P3
Changed lines of the file:
@@
 	1    0    0    -1
 $EndComp
-Text GLabel 4150 7000 0    60   Input ~ 0
+Text GLabel 5400 7050 0    60   Input ~ 0
 SDA
-Text GLabel 4150 6750 0    60   Input ~ 0
+Text GLabel 5400 6800 0    60   Input ~ 0
 SCL
-Text GLabel 3700 7500 0    60   Input ~ 0
+Text GLabel 4950 7550 0    60   Input ~ 0
 +3.3V
-Text GLabel 4150 7250 0    60   Input ~ 0
+Text GLabel 5400 7300 0    60   Input ~ 0
 GND
 $Comp
 L CONN_01X04 P3
 U 1 1 559EA456
-P 4850 7150
-F 0 "P3" H 4850 7400 50  0000 C CNN
-F 1 "CONN_01X04" V 4950 7150 50  0000 C CNN
-F 2 "w_pin_strip:pin_strip_4" H 4850 7150 60  0001 C CNN
-F 3 "" H 4850 7150 60  0000 C CNN
-	1    4850 7150
+P 6100 7200
+F 0 "P3" H 6100 7450 50  0000 C CNN
+F 1 "CONN_01X04" V 6200 7200 50  0000 C CNN
+F 2 "w_pin_strip:pin_strip_4" H 6100 7200 60  0001 C CNN
+F 3 "" H 6100 7200 60  0000 C CNN
+	1    6100 7200
 	1    0    0    -1
 $EndComp
@@
 L GND #PWR07
 U 1 1 559EA7F4
-P 4400 7300
-F 0 "#PWR07" H 4400 7050 50  0001 C CNN
-F 1 "GND" H 4400 7150 50  0000 C CNN
-F 2 "" H 4400 7300 60  0000 C CNN
-F 3 "" H 4400 7300 60  0000 C CNN
-	1    4400 7300
+P 5650 7350
+F 0 "#PWR07" H 5650 7100 50  0001 C CNN
+F 1 "GND" H 5650 7200 50  0000 C CNN
+F 2 "" H 5650 7350 60  0000 C CNN
+F 3 "" H 5650 7350 60  0000 C CNN
+	1    5650 7350
 	1    0    0    -1
 $EndComp
@@
 L +3.3V #PWR08
 U 1 1 559EA8C3
-P 3750 7450
-F 0 "#PWR08" H 3750 7300 50  0001 C CNN
-F 1 "+3.3V" H 3750 7590 50  0000 C CNN
-F 2 "" H 3750 7450 60  0000 C CNN
-F 3 "" H 3750 7450 60  0000 C CNN
-	1    3750 7450
+P 5000 7500
+F 0 "#PWR08" H 5000 7350 50  0001 C CNN
+F 1 "+3.3V" H 5000 7640 50  0000 C CNN
+F 2 "" H 5000 7500 60  0000 C CNN
+F 3 "" H 5000 7500 60  0000 C CNN
+	1    5000 7500
 	1    0    0    -1
 $EndComp
@@
 Connection ~ 3500 5250
 Wire Wire Line
-	4150 7000 4400 7000
-Wire Wire Line
-	4400 7000 4400 7100
-Wire Wire Line
-	4400 7100 4650 7100
-Wire Wire Line
-	4150 6750 4650 6750
-Wire Wire Line
-	4650 6750 4650 7000
-Wire Wire Line
-	4650 7200 4400 7200
-Wire Wire Line
-	4400 7200 4400 7300
-Wire Wire Line
-	4400 7250 4150 7250
-Wire Wire Line
-	4650 7500 4650 7300
-Wire Wire Line
-	3700 7500 4650 7500
-Connection ~ 4400 7250
-Wire Wire Line
-	3750 7450 3750 7500
-Connection ~ 3750 7500
+	5400 7050 5650 7050
+Wire Wire Line
+	5650 6750 5650 7150
+Wire Wire Line
+	5650 7150 5900 7150
+Wire Wire Line
+	5400 6800 5900 6800
+Wire Wire Line
+	5900 6750 5900 7050
+Wire Wire Line
+	5900 7250 5650 7250
+Wire Wire Line
+	5650 7250 5650 7350
+Wire Wire Line
+	5650 7300 5400 7300
+Wire Wire Line
+	5900 7550 5900 7350
+Wire Wire Line
+	4950 7550 5900 7550
+Connection ~ 5650 7300
+Wire Wire Line
+	5000 7500 5000 7550
+Connection ~ 5000 7550
 Wire Wire Line
 	3200 3700 2650 3700
@@
 	2250 3900 1950 3900
 Connection ~ 1950 3900
+$Comp
+L R R1
+U 1 1 5688484C
+P 5650 6600
+F 0 "R1" H 5720 6646 50  0000 L CNN
+F 1 "R" H 5720 6554 50  0000 L CNN
+F 2 "w_smd_resistors:r_0805" V 5580 6600 50  0001 C CNN
+F 3 "" H 5650 6600 50  0000 C CNN
+	1    5650 6600
+	1    0    0    -1
+$EndComp
+$Comp
+L R R2
+U 1 1 568848F5
+P 5900 6600
+F 0 "R2" H 5970 6646 50  0000 L CNN
+F 1 "R" H 5970 6554 50  0000 L CNN
+F 2 "w_smd_resistors:r_0805" V 5830 6600 50  0001 C CNN
+F 3 "" H 5900 6600 50  0000 C CNN
+	1    5900 6600
+	1    0    0    -1
+$EndComp
+Connection ~ 5900 6800
+Connection ~ 5650 7050
+$Comp
+L +3.3V #PWR011
+U 1 1 56884A0A
+P 5750 6350
+F 0 "#PWR011" H 5750 6200 50  0001 C CNN
+F 1 "+3.3V" H 5750 6490 50  0000 C CNN
+F 2 "" H 5750 6350 60  0000 C CNN
+F 3 "" H 5750 6350 60  0000 C CNN
+	1    5750 6350
+	1    0    0    -1
+$EndComp
+Wire Wire Line
+	5900 6450 5900 6400
+Wire Wire Line
+	5900 6400 5650 6400
+Wire Wire Line
+	5650 6400 5650 6450
+Wire Wire Line
+	5750 6350 5750 6400
+Connection ~ 5750 6400
 $EndSCHEMATC
