File: kicad/r-map_v2/breakout_board/temperature_humidity/temperature_humidity.kicad_pcb (KiCad board)
At the start: 2 copper layers, 12.7 x 30.5 mm, 14 parts, among them IC1 ADT7420, P3 CONN_01X04, P4 A0, U1 HIH6100, U2 HIH6100-SOIC8

Commit message: Aggiornamento files gerber e verifica per nuova stampa pcb, revisionate tutte e 4 le board. Il file kicad/r-map_v2/futura_10-2015.zip contiene i files divisi per cartelle di tutte le board
Other:
- board text removed: "Verificare dimensioni package"
Changed lines of the file:
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@@
     (links 24)
     (no_connects 0)
-    (area 108.472857 68.504999 173.1 113.19)
+    (area 144.55 68.504999 160.154686 99.135001)
     (thickness 1.6)
-    (drawings 16)
+    (drawings 11)
     (tracks 128)
     (zones 0)
@@
     (41 Cmts.User user)
     (42 Eco1.User user)
-    (43 Eco2.User user hide)
+    (43 Eco2.User user)
     (44 Edge.Cuts user)
-    (45 Margin user hide)
-    (46 B.CrtYd user hide)
-    (47 F.CrtYd user hide)
-    (48 B.Fab user hide)
-    (49 F.Fab user hide)
+    (45 Margin user)
+    (46 B.CrtYd user)
+    (47 F.CrtYd user)
+    (48 B.Fab user)
+    (49 F.Fab user)
   )
   (setup
@@
     (visible_elements 7FFFFF7F)
     (pcbplotparams
-      (layerselection 0x00030_80000001)
+      (layerselection 0x01030_80000001)
       (usegerberextensions false)
       (excludeedgelayer true)
@@
       (effects (font (size 1 1) (thickness 0.15)) (justify mirror))
     )
-    (fp_text value ADT7420 (at 0 -3.556 180) (layer B.SilkS)
-      (effects (font (size 1 1) (thickness 0.15)) (justify mirror))
+    (fp_text value ADT7420 (at 0 -3.81) (layer B.SilkS) hide
+      (effects (font (size 0.8 1) (thickness 0.15)) (justify mirror))
     )
     (fp_circle (center -1.55 1.55) (end -1.45 1.45) (layer B.SilkS) (width 0.15))
@@
     (effects (font (size 1 1) (thickness 0.2)) (justify mirror))
   )
-  (gr_text "Verificare dimensioni package\n" (at 125.73 87.63) (layer Eco2.User)
-    (effects (font (size 1.5 1.5) (thickness 0.3)))
-  )
   (gr_text rmap.cc (at 146.05 74.93 90) (layer F.SilkS)
     (effects (font (size 1.5 1.5) (thickness 0.3)))
-  )
-  (dimension 30.48 (width 0.3) (layer Eco2.User)
-    (gr_text "30,480 mm" (at 166.45 83.82 270) (layer Eco2.User)
-      (effects (font (size 1.5 1.5) (thickness 0.3)))
-    )
-    (feature1 (pts (xy 157.48 99.06) (xy 167.8 99.06)))
-    (feature2 (pts (xy 157.48 68.58) (xy 167.8 68.58)))
-    (crossbar (pts (xy 165.1 68.58) (xy 165.1 99.06)))
-    (arrow1a (pts (xy 165.1 99.06) (xy 164.513579 97.933496)))
-    (arrow1b (pts (xy 165.1 99.06) (xy 165.686421 97.933496)))
-    (arrow2a (pts (xy 165.1 68.58) (xy 164.513579 69.706504)))
-    (arrow2b (pts (xy 165.1 68.58) (xy 165.686421 69.706504)))
-  )
-  (dimension 12.7 (width 0.3) (layer Eco2.User)
-    (gr_text "12,700 mm" (at 151.13 111.839999) (layer Eco2.User)
-      (effects (font (size 1.5 1.5) (thickness 0.3)))
-    )
-    (feature1 (pts (xy 157.48 99.06) (xy 157.48 113.189999)))
-    (feature2 (pts (xy 144.78 99.06) (xy 144.78 113.189999)))
-    (crossbar (pts (xy 144.78 110.489999) (xy 157.48 110.489999)))
-    (arrow1a (pts (xy 157.48 110.489999) (xy 156.353496 111.07642)))
-    (arrow1b (pts (xy 157.48 110.489999) (xy 156.353496 109.903578)))
-    (arrow2a (pts (xy 144.78 110.489999) (xy 145.906504 111.07642)))
-    (arrow2b (pts (xy 144.78 110.489999) (xy 145.906504 109.903578)))
   )
   (gr_line (start 157.48 99.06) (end 157.48 91.44) (angle 90) (layer Edge.Cuts) (width 0.15))
   (gr_line (start 144.78 99.06) (end 157.48 99.06) (angle 90) (layer Edge.Cuts) (width 0.15))
   (gr_line (start 144.78 91.44) (end 144.78 99.06) (angle 90) (layer Edge.Cuts) (width 0.15))
-  (dimension 26.150901 (width 0.3) (layer F.Fab)
-    (gr_text "26,151 mm" (at 162.014829 86.057127 60.9453959) (layer F.Fab)
-      (effects (font (size 1.5 1.5) (thickness 0.3)))
-    )
-    (feature1 (pts (xy 144.78 91.44) (xy 156.844942 98.142745)))
-    (feature2 (pts (xy 157.48 68.58) (xy 169.544942 75.282745)))
-    (crossbar (pts (xy 167.184717 73.971509) (xy 154.484717 96.831509)))
-    (arrow1a (pts (xy 154.484717 96.831509) (xy 154.519172 95.561976)))
-    (arrow1b (pts (xy 154.484717 96.831509) (xy 155.54442 96.131559)))
-    (arrow2a (pts (xy 167.184717 73.971509) (xy 166.125014 74.671459)))
-    (arrow2b (pts (xy 167.184717 73.971509) (xy 167.150262 75.241042)))
-  )
-  (dimension 22.86 (width 0.3) (layer Margin)
-    (gr_text "22,860 mm" (at 125.650001 80.01 270) (layer Margin)
-      (effects (font (size 1.5 1.5) (thickness 0.3)))
-    )
-    (feature1 (pts (xy 157.48 91.44) (xy 124.300001 91.44)))
-    (feature2 (pts (xy 157.48 68.58) (xy 124.300001 68.58)))
-    (crossbar (pts (xy 127.000001 68.58) (xy 127.000001 91.44)))
-    (arrow1a (pts (xy 127.000001 91.44) (xy 126.41358 90.313496)))
-    (arrow1b (pts (xy 127.000001 91.44) (xy 127.586422 90.313496)))
-    (arrow2a (pts (xy 127.000001 68.58) (xy 126.41358 69.706504)))
-    (arrow2b (pts (xy 127.000001 68.58) (xy 127.586422 69.706504)))
-  )
   (gr_line (start 144.78 68.58) (end 144.78 91.44) (angle 90) (layer Edge.Cuts) (width 0.15))
   (gr_line (start 157.48 68.58) (end 144.78 68.58) (angle 90) (layer Edge.Cuts) (width 0.15))

Commit message: Nuova versione breakout board, inviata a servizio di stampa pcb
Parts:
- added R1: R, w_smd_resistors:r_0805, F.Cu at (155.2, 81.2)
- added R2: R, w_smd_resistors:r_0805, F.Cu at (147.1, 81.2)
- C1: value C -> 0.22uF
- C2, C3: value C -> 0.1uF
- moved C1 2.54 mm to (151.1, 85.1)
- moved C3 2.29 mm to (153.7, 85.1)
- turned IC1 to 180 degrees
Routing:
- net /A1: track 23.2 -> 10.3 mm
- net /A0: track 25.2 -> 12.6 mm, vias 0 -> 2
- net SDA: track 42.0 -> 50.7 mm
- net +3.3V: track 53.1 -> 59.0 mm, vias 0 -> 1
- net GND: track 58.9 -> 54.0 mm
- net SCL: track 36.8 -> 40.2 mm, vias 0 -> 1
- net Net-(C2-Pad1): track 6.16 -> 4.18 mm
Other:
- board text added: "SCL SDA GND VCC"

Commit message: Aggiunti gerber files per breakout board e sistemato case led stima-i2c
Routing:
- added copper zone on B.Cu, net GND
Changed lines of the file:
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@@
   (general
     (links 28)
-    (no_connects 1)
+    (no_connects 0)
     (area 144.704999 68.504999 160.154686 99.135001)
     (thickness 1.6)
@@
       )
     )
+  )
+  (zone (net 2) (net_name GND) (layer B.Cu) (hatch edge 0.508)
+    (connect_pads yes (clearance 0.064))
+    (min_thickness 0.254)
+    (fill yes (arc_segments 16) (thermal_gap 0.508) (thermal_bridge_width 0.508))
+    (polygon
+      (pts
+        (xy 157.0736 98.4504) (xy 145.3896 98.4504) (xy 145.3896 69.1388) (xy 157.0736 69.1388) (xy 157.0736 98.4504)
+      )
+    )
