File: kicad/r-map_v2/i2c_hub/i2c_hub.kicad_pcb (KiCad board)
At the start: 2 copper layers, 142.7 x 21.3 mm, 120 parts, among them J1 RJ45, J2 RJ45, J3 RJ45, J4 RJ45, J5 RJ45, P1 5V, P10 CONN_01X04, P11 5V, P12 SEL, P13 3V3, P14 CONN_01X04, P15 5V, P16 SEL, P17 3V3, P18 CONN_01X04, P19 5V, P2 SEL, P20 SEL, P21 3V3, P23 CONN_01X04, P24 5V, P25 SEL, P27 3V3, P28 5V, P29 SEL, P3 3V3, P30 3V3, P31 5V, P32 SEL, P33 3V3, P34 5V, P35 SEL, P36 3V3, P37 5V, P38 SEL, P39 3V3, P4 CONN_01X04, P42 5V, P43 SEL, P44 3V3, P45 CONN_01X04, P46 5V, P47 SEL, P48 3V3, P49 CONN_01X04, P50 5V, P51 SEL, P52 3V3, P53 CONN_01X04, P55 5V, P56 SEL, P57 3V3, P59 CONN_01X04, P6 5V, P60 5V, P61 SEL, P62 3V3, P63 CONN_01X04, P7 SEL, P8 3V3, U1 LM317_SOT223, U2 LM317_SOT223, U3 ESDA6V1-5SC6, U4 ESDA6V1-5SC6, U5 ESDA6V1-5SC6, U6 ESDA6V1-5SC6

Commit message: modifiche di adeguamento case su stima-th e sistemazione gerber per produzione hub i2c
Parts:
- moved U6 131.3 mm to (38.4, 100.6)
- moved C4 83.6 mm to (62.5, 110.2)
- moved U3 83.5 mm to (169.7, 100.6)
- moved C1 70.7 mm to (145.7, 110.5)
- moved U5 48.3 mm to (86.4, 106.0)
- moved P2 21.8 mm to (173.0, 109.2)
- moved P20 21.8 mm to (151.1, 109.2)
- moved P23 21.8 mm to (151.1, 100.3)
- moved P4 21.8 mm to (173.0, 100.3)
- moved C3 12.8 mm to (75.1, 110.5), turned to 90 degrees
- moved P10 10.2 mm to (166.4, 100.3)
- moved P16 10.2 mm to (156.2, 109.2)
- moved P18 10.2 mm to (156.2, 100.3)
- moved P7 10.2 mm to (166.4, 109.2)
Connections:
- J1 pad 1: Net-(J1-Pad1) -> (no net)
- J1 pad 2: Net-(J1-Pad2) -> (no net)
- J1 pad 7: Net-(J1-Pad7) -> (no net)
- J1 pad 8: Net-(J1-Pad8) -> (no net)
- J2 pad 1: Net-(J2-Pad1) -> (no net)
- J2 pad 2: Net-(J2-Pad2) -> (no net)
- J2 pad 7: Net-(J2-Pad7) -> (no net)
- J2 pad 8: Net-(J2-Pad8) -> (no net)
- J3 pad 1: Net-(J3-Pad1) -> (no net)
- J3 pad 2: Net-(J3-Pad2) -> (no net)
- J3 pad 7: Net-(J3-Pad7) -> (no net)
- J3 pad 8: Net-(J3-Pad8) -> (no net)
- J4 pad 1: Net-(J4-Pad1) -> (no net)
- J4 pad 2: Net-(J4-Pad2) -> (no net)
- J4 pad 7: Net-(J4-Pad7) -> (no net)
- J4 pad 8: Net-(J4-Pad8) -> (no net)
- J5 pad 1: Net-(J5-Pad1) -> (no net)
- J5 pad 2: Net-(J5-Pad2) -> (no net)
- J5 pad 7: Net-(J5-Pad7) -> (no net)
- J5 pad 8: Net-(J5-Pad8) -> (no net)
- U3 pad 3: Net-(U3-Pad3) -> (no net)
- U4 pad 1: /+5V -> /+3.3V
- U4 pad 3: Net-(U4-Pad3) -> (no net)
- U5 pad 3: Net-(U5-Pad3) -> (no net)
- U6 pad 3: Net-(U6-Pad3) -> (no net)
Routing:
- net /+5V: track 299.3 -> 260.0 mm, vias 0 -> 9
- net GND: track 344.4 -> 330.0 mm, vias 11 -> 7
- net /+3.3V: track 259.1 -> 272.0 mm, vias 4 -> 6
- net /SDA: track 169.1 -> 170.9 mm
- net Net-(J4-Pad5): track 7.91 -> 8.69 mm
- added copper zone on B.Cu, net GND
