File: kicad/r-map_v2/breakout_board/Stima_AirQuality_Connector/Stima_AirQuality_Connector.sch (KiCad schematic (older format))
At the start: 5 parts

Commit message: Update schematic for DRC errors
Parts:
- removed U?: Microduino, symbol Microduino
- added U1: Microduino, symbol Microduino
- P1, P2, P3: renamed from P?; footprint (none) -> Pin_Headers:Pin_Header_Straight_1x05_Pitch2.54mm
- P4: renamed from P?; footprint (none) -> Pin_Headers:Pin_Header_Straight_1x04_Pitch2.54mm
Connections:
- net +3V3: now also U1.26 (3V3)
- net +5V: now also U1.27 (5V)
- net CO: now also U1.16 (A1)
- net CO_SCALE_1: now also U1.22 (D10)
- net CO_SCALE_2: now also U1.21 (D11)
- net FET: now also U1.25 (D7)
- net GND: now also U1.1 (GND)
- net NO2: now also U1.17 (A0)
- net NO2_SCALE_1: now also U1.24 (D8)
- net NO2_SCALE_2: now also U1.23 (D9)
- net SCL: now also U1.12 (A5)
- net SDA: now also U1.13 (A4)
Changed lines of the file:
@@
 $EndDescr
 $Comp
-L Microduino U?
-U 1 1 589CCBF6
-P 5200 2750
-F 0 "U?" H 5100 3197 60  0000 C CNN
-F 1 "Microduino" H 5100 3091 60  0000 C CNN
-F 2 "" H 650 -200 60  0000 C CNN
-F 3 "" H 650 -200 60  0000 C CNN
-	1    5200 2750
-	1    0    0    -1
-$EndComp
-$Comp
-L +5V #PWR?
+L +5V #PWR01
 U 1 1 589CCCE0
 P 5950 2450
-F 0 "#PWR?" H -50 -250 50  0001 C CNN
+F 0 "#PWR01" H -50 -250 50  0001 C CNN
 F 1 "+5V" H 5965 2623 50  0000 C CNN
 F 2 "" H -50 -100 50  0001 C CNN
@@
 	5950 2550 5800 2550
 $Comp
-L GND #PWR?
+L GND #PWR02
 U 1 1 589CCCFC
 P 4150 2650
-F 0 "#PWR?" H 0   -150 50  0001 C CNN
+F 0 "#PWR02" H 0   -150 50  0001 C CNN
 F 1 "GND" H 4155 2477 50  0000 C CNN
 F 2 "" H 0   100 50  0001 C CNN
@@
 	4150 2550 4400 2550
 $Comp
-L +3.3V #PWR?
+L +3.3V #PWR03
 U 1 1 589CCD1E
 P 6150 2450
-F 0 "#PWR?" H -50 -600 50  0001 C CNN
+F 0 "#PWR03" H -50 -600 50  0001 C CNN
 F 1 "+3.3V" H 6165 2623 50  0000 C CNN
 F 2 "" H -50 -450 50  0001 C CNN
@@
 	6150 2650 5800 2650
 $Comp
-L CONN_01X05 P?
+L CONN_01X05 P3
 U 1 1 589CCD3F
 P 7650 3200
-F 0 "P?" H 7728 3241 50  0000 L CNN
+F 0 "P3" H 7728 3241 50  0000 L CNN
 F 1 "CONN_01X05" H 7728 3150 50  0000 L CNN
-F 2 "" H 1400 -250 50  0001 C CNN
+F 2 "Pin_Headers:Pin_Header_Straight_1x05_Pitch2.54mm" H 1400 -250 50  0001 C CNN
 F 3 "" H 1400 -250 50  0001 C CNN
 	1    7650 3200
@@
 SDA
 $Comp
-L GND #PWR?
+L GND #PWR04
 U 1 1 589CCDD1
 P 7750 3850
-F 0 "#PWR?" H 7800 3900 50  0001 C CNN
+F 0 "#PWR04" H 7800 3900 50  0001 C CNN
 F 1 "GND" H 7755 3677 50  0000 C CNN
 F 2 "" H 0   -150 50  0001 C CNN
@@
 $EndComp
 $Comp
-L +3.3V #PWR?
+L +3.3V #PWR05
 U 1 1 589CCE09
 P 8050 3350
-F 0 "#PWR?" H 8100 3400 50  0001 C CNN
+F 0 "#PWR05" H 8100 3400 50  0001 C CNN
 F 1 "+3.3V" H 8065 3523 50  0000 C CNN
 F 2 "" H 150 -300 50  0001 C CNN
@@
 	7550 3400 7550 3650
 $Comp
-L +5V #PWR?
+L +5V #PWR06
 U 1 1 589CCE6E
 P 7250 3350
-F 0 "#PWR?" H 7300 3400 50  0001 C CNN
+F 0 "#PWR06" H 7300 3400 50  0001 C CNN
 F 1 "+5V" H 7265 3523 50  0000 C CNN
 F 2 "" H -150 -300 50  0001 C CNN
@@
 	7450 3500 7450 3400
 $Comp
-L CONN_01X05 P?
+L CONN_01X05 P1
 U 1 1 589CCFAB
 P 4100 5350
-F 0 "P?" H 4019 4925 50  0000 C CNN
+F 0 "P1" H 4019 4925 50  0000 C CNN
 F 1 "CONN_01X05" H 4019 5016 50  0000 C CNN
-F 2 "" H -1350 100 50  0001 C CNN
+F 2 "Pin_Headers:Pin_Header_Straight_1x05_Pitch2.54mm" H -1350 100 50  0001 C CNN
 F 3 "" H -1350 100 50  0001 C CNN
 	1    4100 5350
@@
 $EndComp
 $Comp
-L CONN_01X05 P?
+L CONN_01X05 P2
 U 1 1 589CD012
 P 4100 5850
-F 0 "P?" H 4019 5425 50  0000 C CNN
+F 0 "P2" H 4019 5425 50  0000 C CNN
 F 1 "CONN_01X05" H 4019 5516 50  0000 C CNN
-F 2 "" H 0   -50 50  0001 C CNN
+F 2 "Pin_Headers:Pin_Header_Straight_1x05_Pitch2.54mm" H 0   -50 50  0001 C CNN
 F 3 "" H 0   -50 50  0001 C CNN
 	1    4100 5850
@@
 	5550 5750 4300 5750
 $Comp
-L +5V #PWR?
+L +5V #PWR07
 U 1 1 589CD236
 P 5700 5800
-F 0 "#PWR?" H 5750 5850 50  0001 C CNN
+F 0 "#PWR07" H 5750 5850 50  0001 C CNN
 F 1 "+5V" H 5715 5973 50  0000 C CNN
 F 2 "" H -200 -200 50  0001 C CNN
@@
 Wire Wire Line
 	5700 5800 5700 5850
-Wire Wire Line
-	4300 5850 5900 5850
-$Comp
-L GND #PWR?
+$Comp
+L GND #PWR08
 U 1 1 589CD287
 P 5700 6150
-F 0 "#PWR?" H 5750 6200 50  0001 C CNN
+F 0 "#PWR08" H 5750 6200 50  0001 C CNN
 F 1 "GND" H 5705 5977 50  0000 C CNN
 F 2 "" H 1400 200 50  0001 C CNN
@@
 $EndComp
 Wire Wire Line
-	4300 5950 5900 5950
+	4300 5950 5700 5950
 Wire Wire Line
 	5700 5950 5700 6150
-$Comp
-L PWR_FLAG #FLG?
-U 1 1 589CD2EC
-P 5900 5850
-F 0 "#FLG?" H 5950 5900 50  0001 C CNN
-F 1 "PWR_FLAG" V 5900 5978 50  0000 L CNN
-F 2 "" H 50  -50 50  0001 C CNN
-F 3 "" H 50  -50 50  0001 C CNN
-	1    5900 5850
-	0    1    1    0
-$EndComp
-Connection ~ 5700 5850
-$Comp
-L PWR_FLAG #FLG?
-U 1 1 589CD343
-P 5900 5950
-F 0 "#FLG?" H 5950 6000 50  0001 C CNN
-F 1 "PWR_FLAG" V 5900 6078 50  0000 L CNN
-F 2 "" H -50 0   50  0001 C CNN
-F 3 "" H -50 0   50  0001 C CNN
-	1    5900 5950
-	0    1    1    0
-$EndComp
-Connection ~ 5700 5950
 Wire Wire Line
 	4300 6050 5700 6050
 Connection ~ 5700 6050
 $Comp
-L CONN_01X04 P?
+L CONN_01X04 P4
 U 1 1 589CD4E0
 P 7650 4850
-F 0 "P?" V 7650 5150 50  0000 R CNN
+F 0 "P4" V 7650 5150 50  0000 R CNN
 F 1 "CONN_01X04" V 7750 5050 50  0000 R CNN
-F 2 "" H 5750 -250 50  0001 C CNN
+F 2 "Pin_Headers:Pin_Header_Straight_1x04_Pitch2.54mm" H 5750 -250 50  0001 C CNN
 F 3 "" H 5750 -250 50  0001 C CNN
 	1    7650 4850
@@
 TX
 $Comp
-L GND #PWR?
+L GND #PWR09
 U 1 1 589CD795
 P 7700 5250
-F 0 "#PWR?" H 7750 5300 50  0001 C CNN
+F 0 "#PWR09" H 7750 5300 50  0001 C CNN
 F 1 "GND" H 7705 5077 50  0000 C CNN
 F 2 "" H 0   0   50  0001 C CNN
@@
 $EndComp
 $Comp
-L +5V #PWR?
+L +5V #PWR010
 U 1 1 589CD7C2
 P 7950 5050
-F 0 "#PWR?" H 8000 5100 50  0001 C CNN
+F 0 "#PWR010" H 8000 5100 50  0001 C CNN
 F 1 "+5V" H 7965 5223 50  0000 C CNN
 F 2 "" H 100 -200 50  0001 C CNN
@@
 NoConn ~ 4400 2850
 NoConn ~ 4400 2950
+$Comp
+L Microduino U1
+U 1 1 589CF128
+P 5200 2750
+F 0 "U1" H 5100 3197 60  0000 C CNN
+F 1 "Microduino" H 5100 3091 60  0000 C CNN
+F 2 "" H -50 100 60  0000 C CNN
+F 3 "" H -50 100 60  0000 C CNN
+	1    5200 2750
+	1    0    0    -1
+$EndComp
+Wire Wire Line
+	5700 5850 4300 5850
 $EndSCHEMATC

Commit message: complete the NO2-CO boards
Connections:
- net +5V: now also P2.5 (P5); no longer P2.3 (P3)
- net VREF: now reaches U1.18 (REF)
- net VREF: now also P2.3 (P3)
- net CO_SCALE_1: no longer names the net of U1.22 (D10)
- net CO_SCALE_1: no longer P1.2 (P2)
- net CO_SCALE_2: no longer names the net of U1.21 (D11)
- net CO_SCALE_2: no longer P1.3 (P3)
- net FET: no longer names the net of P2.4 (P4)
- net FET: no longer U1.25 (D7)
- net NO2_SCALE_1 renamed SCALE_1
- net SCALE_1: now also P1.2 (P2); no longer P2.5 (P5)
- net NO2_SCALE_2 renamed PWM
- net PWM: now also U1.25 (D7); no longer U1.23 (D9)
- new net SCALE_2: P1.3 (P3), U1.23 (D9)
- no-connect marks 10 -> 13
Changed lines of the file:
@@
 EESchema Schematic File Version 2
+LIBS:Stima_AirQuality_Connector-rescue
 LIBS:power
 LIBS:device
@@
 LIBS:valves
 LIBS:microduino
-EELAYER 26 0
+LIBS:Stima_AirQuality_Connector-cache
+EELAYER 25 0
 EELAYER END
 $Descr A4 11693 8268
@@
 Text GLabel 4800 5050 1    60   Input ~ 0
 CO
-Text GLabel 4950 5050 1    60   Input ~ 0
-CO_SCALE_2
-Text GLabel 5100 5050 1    60   Input ~ 0
-CO_SCALE_1
 Text GLabel 5250 5050 1    60   Input ~ 0
-NO2_SCALE_2
+SCALE_2
 Text GLabel 5400 5050 1    60   Input ~ 0
-NO2_SCALE_1
+SCALE_1
 Text GLabel 5550 5050 1    60   Input ~ 0
-FET
+PWM
 Wire Wire Line
 	4650 5050 4650 5150
@@
 Wire Wire Line
 	4800 5250 4800 5050
-Wire Wire Line
-	4950 5050 4950 5350
-Wire Wire Line
-	4950 5350 4300 5350
-Wire Wire Line
-	4300 5450 5100 5450
-Wire Wire Line
-	5100 5450 5100 5050
-Wire Wire Line
-	5250 5050 5250 5550
-Wire Wire Line
-	5250 5550 4300 5550
-Wire Wire Line
-	4300 5650 5400 5650
-Wire Wire Line
-	5400 5650 5400 5050
-Wire Wire Line
-	5550 5050 5550 5750
-Wire Wire Line
-	5550 5750 4300 5750
 $Comp
 L +5V #PWR07
 U 1 1 589CD236
-P 5700 5800
-F 0 "#PWR07" H 5750 5850 50  0001 C CNN
-F 1 "+5V" H 5715 5973 50  0000 C CNN
-F 2 "" H -200 -200 50  0001 C CNN
-F 3 "" H -200 -200 50  0001 C CNN
-	1    5700 5800
-	1    0    0    -1
-$EndComp
-Wire Wire Line
-	5700 5800 5700 5850
+P 5700 5570
+F 0 "#PWR07" H 5750 5620 50  0001 C CNN
+F 1 "+5V" H 5715 5743 50  0000 C CNN
+F 2 "" H -200 -430 50  0001 C CNN
+F 3 "" H -200 -430 50  0001 C CNN
+	1    5700 5570
+	1    0    0    -1
+$EndComp
 $Comp
 L GND #PWR08
@@
 Wire Wire Line
 	7500 5250 7500 5050
-Text GLabel 6000 3050 2    60   Input ~ 0
-CO_SCALE_1
 Text GLabel 6000 2950 2    60   Input ~ 0
-NO2_SCALE_2
+SCALE_2
 Text GLabel 6000 2850 2    60   Input ~ 0
-NO2_SCALE_1
+SCALE_1
 Text GLabel 6000 2750 2    60   Input ~ 0
-FET
-Text GLabel 6000 3150 2    60   Input ~ 0
-CO_SCALE_2
+PWM
 Wire Wire Line
 	6000 2750 5800 2750
@@
 Wire Wire Line
 	6000 2950 5800 2950
-Wire Wire Line
-	5800 3050 6000 3050
-Wire Wire Line
-	5800 3150 6000 3150
 Text GLabel 5400 3900 3    60   Input ~ 0
 NO2
@@
 	1    0    0    -1
 $EndComp
-Wire Wire Line
-	5700 5850 4300 5850
+Text Label 4450 5450 0    60   ~ 0
+SCALE1
+Text Label 4450 5350 0    60   ~ 0
+SCALE2
+NoConn ~ 5800 3050
+NoConn ~ 5800 3150
+Text GLabel 5500 3900 3    60   Input ~ 0
+VREF
+Wire Wire Line
+	5500 3900 5500 3750
+Wire Wire Line
+	4300 5350 5250 5350
+Wire Wire Line
+	5250 5350 5250 5050
+Wire Wire Line
+	5400 5050 5400 5450
+Wire Wire Line
+	5400 5450 4300 5450
+Wire Wire Line
+	4300 5550 5550 5550
+Wire Wire Line
+	5550 5550 5550 5050
+Wire Wire Line
+	4300 5650 5700 5650
+Wire Wire Line
+	5700 5650 5700 5570
+Text GLabel 4510 5850 2    60   Input ~ 0
+VREF
+Wire Wire Line
+	4510 5850 4300 5850
+NoConn ~ 4300 5750
 $EndSCHEMATC

Commit message: Board correction for MICS-4514 bad pinout. Correction for Stima_AirQuality_Connector connector pinout
Connections:
- net RX: now also U1.9 (RX0)
- net TX: now also U1.8 (TX1)
- no-connect marks 13 -> 15
Changed lines of the file:
@@
 EESchema Schematic File Version 2
-LIBS:Stima_AirQuality_Connector-rescue
 LIBS:power
 LIBS:device
@@
 LIBS:microduino
 LIBS:Stima_AirQuality_Connector-cache
-EELAYER 25 0
+EELAYER 26 0
 EELAYER END
 $Descr A4 11693 8268
@@
 	8050 3350 8050 3500
 Wire Wire Line
-	8050 3500 7850 3500
+	7850 3500 8200 3500
 Wire Wire Line
 	7850 3500 7850 3400
@@
 	7250 3350 7250 3500
 Wire Wire Line
-	7250 3500 7450 3500
+	7170 3500 7450 3500
 Wire Wire Line
 	7450 3500 7450 3400
@@
 	4510 5850 4300 5850
 NoConn ~ 4300 5750
+Text GLabel 4340 3350 0    60   Input ~ 0
+RX
+Wire Wire Line
+	4340 3350 4400 3350
+Text GLabel 4330 3250 0    60   Input ~ 0
+TX
+Wire Wire Line
+	4330 3250 4400 3250
+NoConn ~ 4400 3050
+NoConn ~ 4400 3150
+$Comp
+L PWR_FLAG #FLG011
+U 1 1 591608E3
+P 7170 3500
+F 0 "#FLG011" H 7170 3575 50  0001 C CNN
+F 1 "PWR_FLAG" V 7170 3628 50  0000 L CNN
+F 2 "" H 7170 3500 50  0001 C CNN
+F 3 "" H 7170 3500 50  0001 C CNN
+	1    7170 3500
+	0    -1   -1   0
+$EndComp
+Connection ~ 7250 3500
+$Comp
+L PWR_FLAG #FLG012
+U 1 1 59160B81
+P 8200 3500
+F 0 "#FLG012" H 8200 3575 50  0001 C CNN
+F 1 "PWR_FLAG" V 8200 3628 50  0000 L CNN
+F 2 "" H 8200 3500 50  0001 C CNN
+F 3 "" H 8200 3500 50  0001 C CNN
+	1    8200 3500
+	0    1    1    0
+$EndComp
+Connection ~ 8050 3500
 $EndSCHEMATC
