File: kicad/r-map_v2/microduino_cc1101/microduino_cc1101.sch (KiCad schematic (older format))
At the start: 3 parts, among them J1 Conn_Coaxial, U1 Microduino, U2 CC1101-868MHz-Module

Commit message: Remove unwanted connection for GD02
Unnecessary net remove from schematic and pcb
Connections:
- net labels removed: GD01
- wire segments 28 -> 26
- no-connect marks 19 -> 21
Changed lines of the file:
@@
 Text GLabel 3250 2700 0    60   Input ~ 0
 GDO0
-Text GLabel 3250 2600 0    60   Input ~ 0
-GD01
-Text GLabel 6900 2900 0    60   Input ~ 0
-GD01
-Wire Wire Line
-	6900 2900 7100 2900
 Wire Wire Line
 	7100 2800 6900 2800
-Wire Wire Line
-	3250 2600 3450 2600
 Wire Wire Line
 	3250 2700 3450 2700
@@
 Wire Wire Line
 	4950 2200 4850 2200
+NoConn ~ 7100 2900
+NoConn ~ 3450 2600
 $EndSCHEMATC
