File: kicad/r-map_v2/microduino_lora/microduino_lora.sch (KiCad schematic (older format))
At the start: 3 parts, among them J1 Conn_Coaxial, U1 Microduino, U2 RFM95W-915S2

Commit message: updated schematic of lora shield
Parts:
- removed J1: Conn_Coaxial, lib:SMA_EDGE, symbol Conn_Coaxial
- removed U2: RFM95W-915S2, RF_Modules:Hopref_RFM9XW_SMD, symbol RFM95W-915S2
- added J1: Conn_Coaxial, lib:SMA_EDGE, symbol conn_Coaxial:Conn_Coaxial
- added J2, J3, J4, J5: Conn_01x01, Measurement_Points:Measurement_Point_Round-SMD-Pad_Small, symbol conn_Coaxial:Conn_01x01
- added U2: RFM95, lib:RFM95, symbol lora:RFM95
- U1: footprint Rmap:microduino -> lib:microduino; symbol Microduino -> microduino_lora-rescue:Microduino-RESCUE-microduino_lora
Connections:
- net labels added: FSKTimeOut, RxTimeOut, TxRxDONE
- wire segments 19 -> 31
- no-connect marks 26 -> 20
