File: kicad/stima_devel/microduino_stm32/microduino_stm.sch (KiCad schematic (older format))
At the start: 19 parts, among them IC1 STM32F103CBT6, J1 Conn_01x01, J2 USB_B_Micro, J3 Conn_01x01, SW1 SW_Push, SW2 SW_Push, U1 Microduino, U2 LP2985-3.3, Y1 8M, Y2 32.768KHz cl 12.5pF

Commit message: Change D1 footprint
Parts:
- D1: footprint Diode_SMD:D_SOD-123 -> Diodo:STPS0530Z
- U1: symbol microduino_stm-rescue:Microduino-microduino -> microduino_stm-rescue:Microduino-microduino-microduino_stm-rescue
Changed lines of the file:
@@
 F 0 "D1" V 2054 6130 50  0000 L CNN
 F 1 "D" V 2145 6130 50  0000 L CNN
-F 2 "Diode_SMD:D_SOD-123" H 2100 6050 50  0001 C CNN
+F 2 "Diodo:STPS0530Z" H 2100 6050 50  0001 C CNN
 F 3 "~" H 2100 6050 50  0001 C CNN
 	1    2100 6050
@@
 $EndComp
 $Comp
-L microduino_stm-rescue:Microduino-microduino U1
+L microduino_stm-rescue:Microduino-microduino-microduino_stm-rescue U1
 U 1 1 5FFE8227
 P 9400 2450
