File: kicad/stima_v3/Microduino_ADC_DE/Microduino_ADC_DE.kicad_pcb (KiCad board)
At the start: 2 copper layers, 25.5 x 27.9 mm, 23 parts, among them J1 GS4_b, J2 GS3, J3 GS3, J4 GS3, J5 GS3, J6 GS4_b, J7 GS3, J8 GS3, P1 CONN_1x27, P2 CONN_01X03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

Commit message: reapload kicad scheme
Routing:
- added copper zone on B.Cu, net GND
- added copper zone on F.Cu, net GND
Changed lines of the file:
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@@
-(kicad_pcb (version 20171130) (host pcbnew 5.1.5+dfsg1-2build2)
+(kicad_pcb (version 20171130) (host pcbnew "(5.1.5)-3")
   (general
     (thickness 1.6)
@@
   (segment (start 147.686 82.95) (end 148.236 82.4) (width 0.25) (layer B.Cu) (net 45))
   (segment (start 145.361 82.95) (end 147.686 82.95) (width 0.25) (layer B.Cu) (net 45))
+  (zone (net 24) (net_name GND) (layer B.Cu) (hatch edge 0.508)
+    (connect_pads (clearance 0.35))
+    (min_thickness 0.254)
+    (fill yes (arc_segments 16) (thermal_gap 0.35) (thermal_bridge_width 0.508))
+    (polygon
+      (pts
+        (xy 138.711 90.675) (xy 164.261 90.675) (xy 164.236 62.75) (xy 138.711 62.75)
+      )
+    )
+  )
+  (zone (net 24) (net_name GND) (layer F.Cu) (hatch edge 0.508)
+    (connect_pads (clearance 0.35))
+    (min_thickness 0.254)
+    (fill yes (arc_segments 16) (thermal_gap 0.35) (thermal_bridge_width 0.508))
+    (polygon
+      (pts
+        (xy 138.711 90.675) (xy 164.261 90.675) (xy 164.261 62.75) (xy 138.736 62.75)
+      )
+    )
+  )
 )
