File: kicad/stima_v3/Microduino_BASE_DE/Microduino_Base_DE.sch (KiCad schematic (older format))
At the start: 4 parts, among them P1 CONN_01X02, P2 CONN_01X04, P3 CONN_1x27

Commit message: reapload kicad scheme
Parts:
- added C1: 100nF, Capacitor_SMD:C_0805_2012Metric, symbol Device:C
- added C2, C3: 330uF, Capacitor_Tantalum_SMD:CP_EIA-7343-43_Kemet-X, symbol Device:CP
- added L1: 10uH, SamacSys_Parts:FDSD0630H100MP3, symbol Device:L
- GS1: symbol GS4 -> Libreria_SCH_mia:GS4
- P1: symbol CONN_01X02 -> conn:CONN_01X02
- P2: renamed from P3; symbol CONN_1x27 -> Libreria_SCH_mia:CONN_1x27
- P3: renamed from P2; symbol CONN_01X04 -> conn:CONN_01X04
Connections:
- wire segments 40 -> 60
- no-connect marks 22 -> 20
