File: kicad/stima_v3/Microduino_FT232R_DE/Microduino_FT232R_DE.sch (KiCad schematic (older format))
At the start: 17 parts, among them P1 CONN_1x27, P2 USB_OTG, U1 FT232RL

Commit message: reapload kicad scheme
Parts:
- C1: symbol CP -> Microduino_FT232R_DE-rescue:CP
- C2, C3, C4: symbol C -> Microduino_FT232R_DE-rescue:C
- D1, D2: symbol LED_ALT -> Microduino_FT232R_DE-rescue:LED_ALT
- D3: symbol D_Schottky -> Microduino_FT232R_DE-rescue:D_Schottky
- GS1: symbol GS2 -> Microduino_FT232R_DE-rescue:GS2
- P1: symbol CONN_1x27 -> Microduino_FT232R_DE-rescue:CONN_1x27
- P2: symbol USB_OTG -> Microduino_FT232R_DE-rescue:USB_OTG
- R1, R2, R3, R4, R5, R6: symbol R -> Microduino_FT232R_DE-rescue:R
- U1: symbol FT232RL -> Microduino_FT232R_DE-rescue:FT232RL
Other:
- moved on the sheet: P1
