File: kicad/stima_v3/Microduino_GSM_DE/SIM800C_DE/Microduino_SIM800C_DE.kicad_pcb (KiCad board)
At the start: 2 copper layers, 25.5 x 27.9 mm, 13 parts, among them P1 CONN_1x27, P2 CONN_01X06, U1 SIM800C

Commit message: reapload kicad scheme
Parts:
- ANT1: footprint Libreria_PCB_mia:Molex_SMA_Jack_Edge_Mount_microduino -> Libreria_PCB_mia:Molex_SMA_Jack_Edge_Mount_microduino_2
Connections:
- net /VRTC renamed Net-(P2-Pad2)
Routing:
- net GND: track 98.1 -> 103.8 mm, vias 0 -> 1
