File: kicad/stima_v3/Microduino_GSM_DE/SIM800C_DE/Microduino_SIM800C_DE.sch (KiCad schematic (older format))
At the start: 13 parts, among them P1 CONN_1x27, P2 CONN_01X06, U1 SIM800C

Commit message: reapload kicad scheme
Parts:
- ANT1: footprint Libreria_PCB_mia:Molex_SMA_Jack_Edge_Mount_microduino -> Libreria_PCB_mia:Molex_SMA_Jack_Edge_Mount_microduino_2
Connections:
- net VRTC: no longer names the net of P2.2 (P2)
- no-connect marks 39 -> 40
Changed lines of the file:
@@
 Sheet 1 1
 Title "Microduino SIM800C DE"
-Date "30 giugno 2017"
+Date "24 dicembre 2017"
 Rev "0.0"
 Comp ""
@@
 F 0 "ANT1" H 9250 3100 50  0000 C CNN
 F 1 "CONN_01X02" V 9350 2950 50  0001 C CNN
-F 2 "Libreria_PCB_mia:Molex_SMA_Jack_Edge_Mount_microduino" H 9250 2950 50  0001 C CNN
+F 2 "Libreria_PCB_mia:Molex_SMA_Jack_Edge_Mount_microduino_2" H 9250 2950 50  0001 C CNN
 F 3 "" H 9250 2950 50  0000 C CNN
 	1    9250 2950
@@
 Text Label 2550 4800 0    60   ~ 0
 VBAT
-Text Label 2550 4900 0    60   ~ 0
-VRTC
 Text Label 2550 5000 0    60   ~ 0
 SIM_CLK
@@
 	2550 4800 2250 4800
 Wire Wire Line
-	2250 4900 2550 4900
-Wire Wire Line
 	2550 5000 2250 5000
 Wire Wire Line
@@
 Wire Wire Line
 	4200 3400 4350 3400
-Wire Wire Line
-	6200 1900 6200 2000
 Wire Wire Line
 	6200 1500 6200 1600
@@
 Text Notes 2150 1450 0    99   ~ 20
 GS1 e GS2 saldare i pad 2 e 3 in modo \nda usare i pin D2 (RX1) e D3 (TX1)
+$Comp
+L +3.3V #PWR012
+U 1 1 5A3F6EBF
+P 2250 6150
+F 0 "#PWR012" H 2250 6000 50  0001 C CNN
+F 1 "+3.3V" H 2250 6290 50  0000 C CNN
+F 2 "" H 2250 6150 50  0001 C CNN
+F 3 "" H 2250 6150 50  0001 C CNN
+	1    2250 6150
+	1    0    0    -1
+$EndComp
+$Comp
+L +5V #PWR013
+U 1 1 5A3F6EED
+P 1800 6150
+F 0 "#PWR013" H 1800 6000 50  0001 C CNN
+F 1 "+5V" H 1800 6290 50  0000 C CNN
+F 2 "" H 1800 6150 50  0001 C CNN
+F 3 "" H 1800 6150 50  0001 C CNN
+	1    1800 6150
+	1    0    0    -1
+$EndComp
+$Comp
+L GND #PWR014
+U 1 1 5A3F6F1B
+P 2700 6300
+F 0 "#PWR014" H 2700 6050 50  0001 C CNN
+F 1 "GND" H 2700 6150 50  0000 C CNN
+F 2 "" H 2700 6300 50  0001 C CNN
+F 3 "" H 2700 6300 50  0001 C CNN
+	1    2700 6300
+	1    0    0    -1
+$EndComp
+$Comp
+L PWR_FLAG #FLG015
+U 1 1 5A3F7003
+P 2700 6150
+F 0 "#FLG015" H 2700 6225 50  0001 C CNN
+F 1 "PWR_FLAG" H 2700 6300 50  0000 C CNN
+F 2 "" H 2700 6150 50  0001 C CNN
+F 3 "" H 2700 6150 50  0001 C CNN
+	1    2700 6150
+	1    0    0    -1
+$EndComp
+$Comp
+L PWR_FLAG #FLG016
+U 1 1 5A3F7031
+P 1800 6300
+F 0 "#FLG016" H 1800 6375 50  0001 C CNN
+F 1 "PWR_FLAG" H 1800 6450 50  0000 C CNN
+F 2 "" H 1800 6300 50  0001 C CNN
+F 3 "" H 1800 6300 50  0001 C CNN
+	1    1800 6300
+	-1   0    0    1
+$EndComp
+$Comp
+L PWR_FLAG #FLG017
+U 1 1 5A3F705F
+P 2250 6300
+F 0 "#FLG017" H 2250 6375 50  0001 C CNN
+F 1 "PWR_FLAG" H 2250 6450 50  0000 C CNN
+F 2 "" H 2250 6300 50  0001 C CNN
+F 3 "" H 2250 6300 50  0001 C CNN
+	1    2250 6300
+	-1   0    0    1
+$EndComp
+Wire Wire Line
+	2700 6150 2700 6300
+Wire Wire Line
+	2250 6150 2250 6300
+Wire Wire Line
+	1800 6150 1800 6300
+Wire Wire Line
+	6200 1900 6200 2000
+NoConn ~ 2250 4900
+$Comp
+L PWR_FLAG #FLG018
+U 1 1 5A3F9F08
+P 3150 6300
+F 0 "#FLG018" H 3150 6375 50  0001 C CNN
+F 1 "PWR_FLAG" H 3150 6450 50  0000 C CNN
+F 2 "" H 3150 6300 50  0001 C CNN
+F 3 "" H 3150 6300 50  0001 C CNN
+	1    3150 6300
+	-1   0    0    1
+$EndComp
+Text Label 3150 6050 0    60   ~ 0
+VBAT
+Wire Wire Line
+	3150 6050 3150 6300
 $EndSCHEMATC
