File: kicad/stima_v3/Microduino_GSM_DE/SIM_shield_DE/Microduino_SIM_shield_DE.kicad_pcb (KiCad board)
At the start: 2 copper layers, 25.5 x 27.9 mm, 20 parts, among them P1 CONN_1x27, P2 CONN_01X06, U1 TLV62569, U2 ESDA6V1-5W6

Commit message: reapload kicad scheme
Routing:
- net GND: track 134.4 -> 124.5 mm
Changed lines of the file:
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@@
     (thickness 1.6)
     (drawings 29)
-    (tracks 171)
+    (tracks 166)
     (zones 0)
     (modules 20)
@@
   (title_block
     (title "Microduino SIM shield DE")
-    (date "04 dicembre 2017")
+    (date "24 dicembre 2017")
     (rev 2.0)
   )
@@
   )
   (setup
-    (last_trace_width 0.25)
+    (last_trace_width 0.5)
     (user_trace_width 0.4)
     (user_trace_width 0.5)
@@
   )
   (module Libreria_PCB_mia:mini_sim_card_holder (layer B.Cu)
-    (at 151.431 77.245 180)
+    (at 151.411 77.225 180)
     (tags SIM)
     (attr smd)
@@
     (pad 6 thru_hole circle (at 0 -12.7 90) (size 2.1 2.1) (drill 1.5) (layers *.Cu *.Mask)
       (net 29 /VSIM))
-    (model ${KISYS3DMOD}/Pin_Headers.3dshapes/Pin_Header_Straight_1x06_Pitch2.54mm.wrl
-      (at (xyz 0 -0.25 0))
-      (scale (xyz 1 1 1))
-      (rotate (xyz 0 0 90))
-    )
   )
   (module TO_SOT_Packages_SMD:SOT-363_SC-70-6 (layer F.Cu)
@@
     (descr "Through hole straight socket strip, 1x09, 2.54mm pitch, single row")
     (tags "Through hole socket strip THT 1x09 2.54mm single row")
-    (fp_text reference P1 (at 3.16 -1.79 180) (layer B.SilkS)
+    (fp_text reference P1 (at 2.26 -1.56 180) (layer B.SilkS)
       (effects (font (size 1 1) (thickness 0.15)) (justify mirror))
     )
@@
     (pad 27 thru_hole circle (at 20.32 0 180) (size 2.1 2.1) (drill 1.5) (layers *.Cu *.Mask)
       (net 24 GND))
-    (model ${KISYS3DMOD}/Socket_Strips.3dshapes/Socket_Strip_Straight_1x09_Pitch2.54mm.wrl
-      (at (xyz 0 -0.4 0))
-      (scale (xyz 1 1 1))
-      (rotate (xyz 0 0 270))
-    )
   )
   (module Resistors_SMD:R_0805 (layer F.Cu)
@@
     (tags "capacitor 0805")
     (attr smd)
-    (fp_text reference C2 (at 2.04 1.82 360) (layer F.SilkS)
+    (fp_text reference C2 (at 1.81 1.84 360) (layer F.SilkS)
       (effects (font (size 1 1) (thickness 0.15)))
     )
@@
       (effects (font (size 1 1) (thickness 0.15)))
     )
-    (fp_text user %R (at 2.04 1.82 360) (layer F.Fab)
+    (fp_text user %R (at 1.81 1.84 360) (layer F.Fab)
       (effects (font (size 1 1) (thickness 0.15)))
     )
@@
   (segment (start 160.601 88.165) (end 161.571 88.165) (width 0.75) (layer F.Cu) (net 1))
   (segment (start 160.601 88.165) (end 161.571 88.165) (width 0.75) (layer F.Cu) (net 1))
+  (segment (start 150.571 88.635) (end 150.571 89.875) (width 0.5) (layer F.Cu) (net 24))
+  (segment (start 147.411 88.825) (end 148.461 89.875) (width 0.75) (layer F.Cu) (net 24))
+  (segment (start 154.441 89.875) (end 155.451 88.865) (width 0.75) (layer F.Cu) (net 24))
+  (segment (start 148.461 89.875) (end 150.571 89.875) (width 0.75) (layer F.Cu) (net 24))
+  (segment (start 150.571 89.875) (end 154.441 89.875) (width 0.75) (layer F.Cu) (net 24))
   (segment (start 144.821 79.525) (end 144.821 87.765) (width 1) (layer F.Cu) (net 24))
   (segment (start 144.151 79.525) (end 143.511 79.525) (width 1) (layer F.Cu) (net 24))
@@
   (segment (start 144.631 87.775) (end 144.151 87.295) (width 1) (layer F.Cu) (net 24))
   (segment (start 144.151 87.295) (end 144.151 79.525) (width 1) (layer F.Cu) (net 24))
-  (segment (start 155.331 85.045) (end 156.451 85.045) (width 0.5) (layer B.Cu) (net 24))
-  (segment (start 157.761 89.975) (end 157.761 88.865) (width 0.5) (layer F.Cu) (net 24))
-  (segment (start 157.701 90.035) (end 157.761 89.975) (width 0.5) (layer F.Cu) (net 24))
-  (via (at 157.701 90.035) (size 1) (drill 0.5) (layers F.Cu B.Cu) (net 24))
-  (segment (start 157.701 86.295) (end 157.701 90.035) (width 0.5) (layer B.Cu) (net 24))
+  (segment (start 155.331 85.045) (end 156.451 85.045) (width 0.5) (layer B.Cu) (net 24) (status 10))
+  (segment (start 157.771 89.715) (end 157.761 88.865) (width 0.5) (layer F.Cu) (net 24))
+  (segment (start 157.711 89.775) (end 157.771 89.715) (width 0.5) (layer F.Cu) (net 24))
+  (via (at 157.711 89.775) (size 1) (drill 0.5) (layers F.Cu B.Cu) (net 24))
+  (segment (start 157.701 86.295) (end 157.711 89.775) (width 0.5) (layer B.Cu) (net 24))
   (segment (start 156.451 85.045) (end 157.701 86.295) (width 0.5) (layer B.Cu) (net 24))
   (segment (start 151.351 79.525) (end 152.941 79.525) (width 1) (layer F.Cu) (net 24))
   (segment (start 152.941 79.525) (end 153.441 80.025) (width 1) (layer F.Cu) (net 24))
-  (segment (start 155.331 85.045) (end 155.331 80.425) (width 0.5) (layer B.Cu) (net 24))
+  (segment (start 155.331 85.045) (end 155.331 80.425) (width 0.5) (layer B.Cu) (net 24) (status 10))
   (segment (start 153.441 78.535) (end 153.441 80.025) (width 0.25) (layer F.Cu) (net 24))
   (segment (start 152.801 77.895) (end 153.441 78.535) (width 0.5) (layer F.Cu) (net 24))
@@
   (segment (start 153.441 79.015) (end 155.486 76.975) (width 1) (layer F.Cu) (net 24))
   (segment (start 153.441 80.025) (end 153.271 80.025) (width 0.5) (layer F.Cu) (net 24) (status 30))
-  (segment (start 155.451 88.865) (end 155.451 89.575) (width 0.4) (layer F.Cu) (net 24))
-  (segment (start 155.451 89.575) (end 155.031 89.995) (width 0.4) (layer F.Cu) (net 24))
-  (segment (start 148.581 89.995) (end 147.411 88.825) (width 0.4) (layer F.Cu) (net 24))
-  (segment (start 155.031 89.995) (end 148.581 89.995) (width 0.4) (layer F.Cu) (net 24))
   (segment (start 147.411 88.825) (end 143.691 88.825) (width 0.4) (layer F.Cu) (net 24))
   (segment (start 143.691 88.825) (end 143.031 88.165) (width 0.4) (layer F.Cu) (net 24))
   (segment (start 143.031 88.165) (end 141.251 88.165) (width 0.4) (layer F.Cu) (net 24))
   (segment (start 155.451 88.865) (end 157.761 88.865) (width 1) (layer F.Cu) (net 24))
-  (segment (start 154.821 90.025) (end 155.001 90.025) (width 1) (layer F.Cu) (net 24))
-  (segment (start 150.571 90.025) (end 154.821 90.025) (width 1) (layer F.Cu) (net 24))
-  (segment (start 155.001 90.025) (end 155.451 89.575) (width 1) (layer F.Cu) (net 24))
   (segment (start 145.631 81.135) (end 145.741 81.135) (width 1) (layer F.Cu) (net 24))
   (segment (start 145.741 81.135) (end 147.351 79.525) (width 1) (layer F.Cu) (net 24))
@@
   (segment (start 147.351 79.525) (end 145.631 79.525) (width 1) (layer F.Cu) (net 24))
   (segment (start 145.631 81.135) (end 145.631 79.525) (width 1) (layer F.Cu) (net 24))
-  (segment (start 150.571 88.635) (end 150.571 90.025) (width 0.5) (layer F.Cu) (net 24))
   (segment (start 147.411 88.825) (end 147.491 88.825) (width 1) (layer F.Cu) (net 24))
-  (segment (start 147.491 88.825) (end 148.691 90.025) (width 1) (layer F.Cu) (net 24))
-  (segment (start 148.691 90.025) (end 150.571 90.025) (width 1) (layer F.Cu) (net 24))
   (segment (start 147.411 88.825) (end 143.691 88.825) (width 1) (layer F.Cu) (net 24))
   (segment (start 143.691 88.825) (end 143.031 88.165) (width 1) (layer F.Cu) (net 24))
@@
   (segment (start 158.136 68.22) (end 157.761 67.845) (width 1) (layer F.Cu) (net 25))
   (via (at 146.461 76.865) (size 1) (drill 0.5) (layers F.Cu B.Cu) (net 26))
-  (segment (start 150.251 71.945) (end 150.251 73.075) (width 0.5) (layer B.Cu) (net 26))
+  (segment (start 150.251 71.945) (end 150.251 73.075) (width 0.5) (layer B.Cu) (net 26) (status 10))
   (segment (start 150.251 73.075) (end 146.461 76.865) (width 0.5) (layer B.Cu) (net 26))
   (segment (start 144.401 74.805) (end 144.401 75.855) (width 0.4) (layer F.Cu) (net 26))
@@
   (segment (start 150.786 75.1) (end 150.781 75.105) (width 0.5) (layer F.Cu) (net 27))
   (via (at 150.781 75.105) (size 1) (drill 0.5) (layers F.Cu B.Cu) (net 27))
-  (segment (start 150.251 75.635) (end 150.251 85.045) (width 0.5) (layer B.Cu) (net 27))
+  (segment (start 150.251 75.635) (end 150.251 85.045) (width 0.5) (layer B.Cu) (net 27) (status 20))
   (segment (start 150.781 75.105) (end 150.251 75.635) (width 0.5) (layer B.Cu) (net 27))
   (segment (start 151.471 72.855) (end 151.471 74.415) (width 0.5) (layer F.Cu) (net 27))
@@
   (segment (start 152.291 71.885) (end 152.961 71.215) (width 0.5) (layer F.Cu) (net 28))
   (segment (start 152.961 70.555) (end 152.961 70.785) (width 0.5) (layer F.Cu) (net 28))
-  (segment (start 152.791 70.665) (end 152.791 71.945) (width 0.5) (layer B.Cu) (net 28))
+  (segment (start 152.791 70.665) (end 152.791 71.945) (width 0.5) (layer B.Cu) (net 28) (status 20))
   (via (at 152.961 70.555) (size 1) (drill 0.5) (layers F.Cu B.Cu) (net 28))
   (segment (start 152.961 70.555) (end 152.791 70.665) (width 0.5) (layer B.Cu) (net 28))
@@
   (via (at 146.421 69.405) (size 1) (drill 0.5) (layers F.Cu B.Cu) (net 29))
   (segment (start 155.331 70.645) (end 154.071 69.385) (width 0.4) (layer B.Cu) (net 29))
-  (segment (start 155.331 71.945) (end 155.331 70.645) (width 0.4) (layer B.Cu) (net 29))
+  (segment (start 155.331 71.945) (end 155.331 70.645) (width 0.4) (layer B.Cu) (net 29) (status 10))
   (segment (start 146.301 73.505) (end 146.301 70.965) (width 0.4) (layer F.Cu) (net 29))
   (segment (start 145.061 68.755) (end 146.076 69.77) (width 0.5) (layer F.Cu) (net 29))
