File: kicad/stima_v3/Microduino_GSM_DE/SIM_shield_DE/Microduino_SIM_shield_DE.sch (KiCad schematic (older format))
At the start: 20 parts, among them P1 CONN_1x27, P2 CONN_01X06, U1 TLV62569, U2 ESDA6V1-5W6

Commit message: reapload kicad scheme
Parts:
- C1, C2, C3, C4, C5, C8: symbol C -> Device:C
- C6, C7: symbol CP -> Device:CP
- L1: symbol L -> Device:L
- P1: symbol CONN_1x27 -> Libreria_SCH_mia:CONN_1x27
- P2: symbol CONN_01X06 -> conn:CONN_01X06
- R1, R2, R3, R4, R5, R6: symbol R -> Device:R
- SIM1: symbol SIM-CARD -> Libreria_SCH_mia:SIM-CARD
- U1: symbol TLV62569 -> Libreria_SCH_mia:TLV62569
- U2: symbol ESDA6V1-5W6 -> Libreria_SCH_mia:ESDA6V1-5W6
Connections:
- wire segments 78 -> 93
Changed lines of the file:
@@
-EESchema Schematic File Version 2
-LIBS:Libreria_SCH_mia
-LIBS:power
-LIBS:device
-LIBS:transistors
-LIBS:conn
-LIBS:linear
-LIBS:regul
-LIBS:74xx
-LIBS:cmos4000
-LIBS:adc-dac
-LIBS:memory
-LIBS:xilinx
-LIBS:microcontrollers
-LIBS:dsp
-LIBS:microchip
-LIBS:analog_switches
-LIBS:motorola
-LIBS:texas
-LIBS:intel
-LIBS:audio
-LIBS:interface
-LIBS:digital-audio
-LIBS:philips
-LIBS:display
-LIBS:cypress
-LIBS:siliconi
-LIBS:opto
-LIBS:atmel
-LIBS:contrib
-LIBS:valves
-LIBS:Microduino_SIM_shield_DE-cache
-EELAYER 25 0
+EESchema Schematic File Version 4
+EELAYER 30 0
 EELAYER END
 $Descr A4 11693 8268
@@
 Sheet 1 1
 Title "Microduino SIM shield DE"
-Date "04 dicembre 2017"
+Date "24 dicembre 2017"
 Rev "2.0"
 Comp ""
@@
 NoConn ~ 3850 2600
 $Comp
-L GND #PWR01
+L power:GND #PWR01
 U 1 1 58D4FFFC
 P 3600 2850
@@
 $EndComp
 $Comp
-L +5V #PWR02
+L power:+5V #PWR02
 U 1 1 58D50BEE
 P 1650 2700
@@
 $EndComp
 $Comp
-L +3.3V #PWR03
+L power:+3.3V #PWR03
 U 1 1 58D50CA7
 P 1650 2600
@@
 UPIN 27
 $Comp
-L CONN_1x27 P1
+L Libreria_SCH_mia:CONN_1x27 P1
 U 1 1 58E8C7EF
 P 2300 2700
@@
 NoConn ~ 1850 2400
 $Comp
-L CONN_01X06 P2
+L conn:CONN_01X06 P2
 U 1 1 59500203
 P 3050 4350
@@
 VSIM
 $Comp
-L GND #PWR04
+L power:GND #PWR04
 U 1 1 59504B94
 P 6850 2850
@@
 $EndComp
 $Comp
-L GND #PWR05
+L power:GND #PWR05
 U 1 1 59504BBA
 P 9200 2850
@@
 NoConn ~ 3850 1900
 $Comp
-L C C8
+L Device:C C8
 U 1 1 5968D92E
 P 3400 5050
@@
 $EndComp
 $Comp
-L GND #PWR06
+L power:GND #PWR06
 U 1 1 5968D961
 P 3400 5450
@@
 $EndComp
 $Comp
-L R R3
+L Device:R R3
 U 1 1 5968E007
 P 7400 2400
@@
 $EndComp
 $Comp
-L R R1
+L Device:R R1
 U 1 1 5968E044
 P 6850 2650
@@
 $EndComp
 $Comp
-L GND #PWR07
+L power:GND #PWR07
 U 1 1 5968E3F5
 P 4900 2850
@@
 $EndComp
 $Comp
-L +5V #PWR08
+L power:+5V #PWR08
 U 1 1 5968E56D
 P 4550 2000
@@
 $EndComp
 $Comp
-L R R4
+L Device:R R4
 U 1 1 5968EC42
 P 3550 4300
@@
 $EndComp
 $Comp
-L R R5
+L Device:R R5
 U 1 1 5968ECA3
 P 3550 4400
@@
 $EndComp
 $Comp
-L R R6
+L Device:R R6
 U 1 1 5968ECD2
 P 3550 4500
@@
 	4700 4100 3250 4100
 Wire Wire Line
-	3700 4300 4700 4300
-Wire Wire Line
-	3700 4400 4700 4400
-Wire Wire Line
-	3700 4500 4700 4500
-Wire Wire Line
-	3250 4600 4700 4600
+	3700 4300 4100 4300
+Wire Wire Line
+	3700 4400 4200 4400
+Wire Wire Line
+	3700 4500 4300 4500
+Wire Wire Line
+	3250 4600 3400 4600
 Wire Wire Line
 	6850 2800 6850 2850
@@
 Connection ~ 7600 2000
 Wire Wire Line
-	6700 2400 6900 2400
+	6700 2400 6850 2400
 Wire Wire Line
 	6850 2400 6850 2500
 Connection ~ 6850 2400
 Wire Wire Line
-	4550 2000 5700 2000
+	4550 2000 4900 2000
 Wire Wire Line
 	4900 2000 4900 2300
@@
 	4200 5400 4200 5450
 $Comp
-L GND #PWR09
+L power:GND #PWR09
 U 1 1 59690EA6
 P 4200 5450
@@
 $EndComp
 $Comp
-L GND #PWR010
+L power:GND #PWR010
 U 1 1 596919DD
 P 8900 4400
@@
 Connection ~ 9200 2000
 $Comp
-L ESDA6V1-5W6 U2
+L Libreria_SCH_mia:ESDA6V1-5W6 U2
 U 1 1 596937F2
 P 4200 5050
@@
 $EndComp
 $Comp
-L SIM-CARD SIM1
+L Libreria_SCH_mia:SIM-CARD SIM1
 U 1 1 59693AB0
 P 8300 4300
@@
 $EndComp
 $Comp
-L CP C7
+L Device:CP C7
 U 1 1 598C1A9F
 P 9600 2450
@@
 	9600 2600 9600 2850
 $Comp
-L CP C6
+L Device:CP C6
 U 1 1 598C1AF0
 P 9200 2450
@@
 Connection ~ 9600 2000
 $Comp
-L GND #PWR011
+L power:GND #PWR011
 U 1 1 598C1C9A
 P 9600 2850
@@
 VSIM = 1,8 volt
 $Comp
-L TLV62569 U1
+L Libreria_SCH_mia:TLV62569 U1
 U 1 1 59ACD115
 P 6200 2200
@@
 Connection ~ 5650 2000
 Wire Wire Line
-	7250 2000 9900 2000
+	7250 2000 7600 2000
 Wire Wire Line
 	6200 2700 6200 2850
 $Comp
-L GND #PWR012
+L power:GND #PWR012
 U 1 1 59ACD5B2
 P 6200 2850
@@
 $EndComp
 $Comp
-L L L1
+L Device:L L1
 U 1 1 59ACD613
 P 7100 2000
@@
 	6700 2000 6950 2000
 $Comp
-L C C1
+L Device:C C1
 U 1 1 5A259459
 P 4900 2450
@@
 $EndComp
 $Comp
-L C C4
+L Device:C C4
 U 1 1 5A2594E6
 P 8400 2450
@@
 $EndComp
 $Comp
-L C C5
+L Device:C C5
 U 1 1 5A25A485
 P 8800 2450
@@
 	8400 2600 8400 2850
 $Comp
-L GND #PWR013
+L power:GND #PWR013
 U 1 1 5A25AD2E
 P 8800 2850
@@
 $EndComp
 $Comp
-L GND #PWR014
+L power:GND #PWR014
 U 1 1 5A25AD6C
 P 8400 2850
@@
 	7250 2400 7200 2400
 $Comp
-L R R2
+L Device:R R2
 U 1 1 5A25B1F9
 P 7050 2400
@@
 NoConn ~ 3250 4200
 $Comp
-L PWR_FLAG #FLG015
+L power:PWR_FLAG #FLG015
 U 1 1 5A25BD85
 P 8300 5650
@@
 $EndComp
 $Comp
-L PWR_FLAG #FLG016
+L power:PWR_FLAG #FLG016
 U 1 1 5A25BEA1
 P 7800 5650
@@
 $EndComp
 $Comp
-L PWR_FLAG #FLG017
+L power:PWR_FLAG #FLG017
 U 1 1 5A25C0A7
 P 8800 5500
@@
 $EndComp
 $Comp
-L GND #PWR018
+L power:GND #PWR018
 U 1 1 5A25C19E
 P 8800 5650
@@
 $EndComp
 $Comp
-L +3V3 #PWR019
+L power:+3V3 #PWR019
 U 1 1 5A25C590
 P 8300 5500
@@
 $EndComp
 $Comp
-L +5V #PWR020
+L power:+5V #PWR020
 U 1 1 5A25C5C8
 P 7800 5500
@@
 	8800 5500 8800 5650
 $Comp
-L C C2
+L Device:C C2
 U 1 1 5A26B13D
 P 5300 2450
@@
 	5300 2600 5300 2850
 $Comp
-L GND #PWR021
+L power:GND #PWR021
 U 1 1 5A26B2D9
 P 5300 2850
@@
 $EndComp
 $Comp
-L C C3
+L Device:C C3
 U 1 1 5A26B420
 P 8000 2450
@@
 $EndComp
 $Comp
-L GND #PWR022
+L power:GND #PWR022
 U 1 1 5A26B466
 P 8000 2850
@@
 Wire Wire Line
 	8000 2600 8000 2850
+Wire Wire Line
+	4900 2000 5300 2000
+Wire Wire Line
+	3400 4600 4400 4600
+Wire Wire Line
+	7600 2000 8000 2000
+Wire Wire Line
+	6850 2400 6900 2400
+Wire Wire Line
+	4400 4600 4700 4600
+Wire Wire Line
+	4300 4500 4700 4500
+Wire Wire Line
+	4200 4400 4700 4400
+Wire Wire Line
+	4100 4300 4700 4300
+Wire Wire Line
+	9200 2000 9600 2000
+Wire Wire Line
+	9600 2000 9900 2000
+Wire Wire Line
+	5650 2000 5700 2000
+Wire Wire Line
+	8400 2000 8800 2000
+Wire Wire Line
+	8800 2000 9200 2000
+Wire Wire Line
+	5300 2000 5650 2000
+Wire Wire Line
+	8000 2000 8400 2000
 $EndSCHEMATC
