File: kicad/stima_v3/Microduino_HUB_DE/Microduino_HUB_DE.sch (KiCad schematic (older format))
At the start: 54 parts, among them P1 CONN_01X04, P2 CONN_01X04, P3 CONN_01X04, P4 USB_B, P5 CONN_01X04, P6 CONN_01X04, P7 CONN_01X04, P8 CONN_01X04, U1 PCA9517A, U2 PCA9517A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

Commit message: reapload kicad scheme
Parts:
- C1, C10, C11, C12, C15, C2, C3, C4, C5, C6, C7, C8, C9: symbol C -> Microduino_HUB_DE-rescue:C
- C13, C14: symbol CP -> Microduino_HUB_DE-rescue:CP
- D1: symbol D_Schottky -> Microduino_HUB_DE-rescue:D_Schottky
- GS1, GS2, GS3, GS4, GS5, GS6: symbol GS3 -> Microduino_HUB_DE-rescue:GS3
- L1: symbol L -> Microduino_HUB_DE-rescue:L
- P1, P2, P3, P5, P6, P7, P8: symbol CONN_01X04 -> Microduino_HUB_DE-rescue:CONN_01X04
- P4: symbol USB_B-RESCUE-Microduino_HUB_DE -> Microduino_HUB_DE-rescue:USB_B-RESCUE-Microduino_HUB_DE
- R1, R10, R11, R12, R13, R14, R15, R16, R2, R3, R4, R5, R6, R7, R8, R9: symbol R -> Microduino_HUB_DE-rescue:R
- U1, U2, U3, U4, U6, U7: symbol PCA9517 -> Microduino_HUB_DE-rescue:PCA9517
- U5: symbol TLV62569 -> Microduino_HUB_DE-rescue:TLV62569
Other:
- moved on the sheet: C13, C14, C15, D1, L1, P4, R15, R16, U5
