File: kicad/stima_v3/Microduino_OPC_DE/Microduino_OPC_DE.kicad_pcb (KiCad board)
At the start: 2 copper layers, 25.5 x 27.9 mm, 10 parts, among them J1 CONN_01X06, J2 GS3, P1 CONN_1x27, Q1 BSP315PH6327XTSA1, Q2 BC847B, U1 MAX3378E

Commit message: reapload kicad scheme
Connections:
- R3 pad 1: Net-(J1-Pad1) -> +5V
Routing:
- net +5V: track 27.9 -> 50.0 mm, vias 1 -> 2
- net Net-(J1-Pad1): track 20.2 -> 7.80 mm, vias 2 -> 1
- net GND: track 32.3 -> 40.0 mm
- net Net-(J1-Pad4): track 19.7 -> 23.3 mm, vias 0 -> 2
- net Net-(J1-Pad5): track 18.4 -> 20.6 mm
- net D6: track 26.4 -> 28.1 mm
- net Net-(J1-Pad2): track 22.1 -> 21.6 mm, vias 0 -> 2
- net Net-(J1-Pad3): track 20.9 -> 21.0 mm, vias 0 -> 2
- added copper zone on B.Cu, net GND
- added copper zone on F.Cu, net GND
