File: kicad/stima_v3/Microduino_OPC_DE/Microduino_OPC_DE.sch (KiCad schematic (older format))
At the start: 10 parts, among them J1 CONN_01X06, J2 GS3, P1 CONN_1x27, Q1 BSP315PH6327XTSA1, Q2 BC847B, U1 MAX3378E

Commit message: reapload kicad scheme
Parts:
- J1: symbol CONN_01X06 -> conn:CONN_01X06
- J2: symbol GS3 -> conn:GS3
- P1: symbol CONN_1x27 -> Libreria_SCH_mia1:CONN_1x27
- Q1: symbol Q_PMOS_GDS -> Device:Q_PMOS_GDS
- Q2: symbol Q_NPN_BEC -> Device:Q_NPN_BEC
- R1, R2, R3, R4: symbol R -> Device:R
- U1: symbol MAX3378E -> Libreria_SCH_mia1:MAX3378E
Connections:
- wire segments 70 -> 72
Changed lines of the file:
@@
-EESchema Schematic File Version 2
-LIBS:Libreria_SCH_mia
-LIBS:power
-LIBS:device
-LIBS:transistors
-LIBS:conn
-LIBS:linear
-LIBS:regul
-LIBS:74xx
-LIBS:cmos4000
-LIBS:adc-dac
-LIBS:memory
-LIBS:xilinx
-LIBS:microcontrollers
-LIBS:dsp
-LIBS:microchip
-LIBS:analog_switches
-LIBS:motorola
-LIBS:texas
-LIBS:intel
-LIBS:audio
-LIBS:interface
-LIBS:digital-audio
-LIBS:philips
-LIBS:display
-LIBS:cypress
-LIBS:siliconi
-LIBS:opto
-LIBS:atmel
-LIBS:contrib
-LIBS:valves
-LIBS:Microduino_OPC_DE-cache
-EELAYER 25 0
+EESchema Schematic File Version 4
+EELAYER 30 0
 EELAYER END
 $Descr A4 11693 8268
@@
 Sheet 1 1
 Title "Microduino OPC DE"
-Date "07 aprile 2014"
+Date "03 novembre 2019"
 Rev "0.0"
 Comp ""
@@
 NoConn ~ 8250 3700
 $Comp
-L GND #PWR01
+L power:GND #PWR01
 U 1 1 58D4FFFC
 P 8000 3950
@@
 $EndComp
 $Comp
-L +5V #PWR02
+L power:+5V #PWR02
 U 1 1 58D50BEE
 P 5850 3800
@@
 $EndComp
 $Comp
-L +3.3V #PWR03
+L power:+3.3V #PWR03
 U 1 1 58D50CA7
 P 6050 3700
@@
 UPIN 27
 $Comp
-L CONN_1x27 P1
+L Libreria_SCH_mia1:CONN_1x27 P1
 U 1 1 58E8C7EF
 P 6700 3800
@@
 +5V
 $Comp
-L +3.3V #PWR04
+L power:+3.3V #PWR04
 U 1 1 5A3F7B13
 P 6700 5000
@@
 $EndComp
 $Comp
-L +5V #PWR05
+L power:+5V #PWR05
 U 1 1 5A3F7B2B
 P 7250 5000
@@
 $EndComp
 $Comp
-L GND #PWR06
+L power:GND #PWR06
 U 1 1 5A3F7B43
 P 7800 5200
@@
 $EndComp
 $Comp
-L PWR_FLAG #FLG07
+L power:PWR_FLAG #FLG07
 U 1 1 5A3F7B5B
 P 7800 5000
@@
 $EndComp
 $Comp
-L PWR_FLAG #FLG08
+L power:PWR_FLAG #FLG08
 U 1 1 5A3F7B73
 P 7250 5200
@@
 $EndComp
 $Comp
-L PWR_FLAG #FLG09
+L power:PWR_FLAG #FLG09
 U 1 1 5A3F7B8B
 P 6700 5200
@@
 	8000 3800 7900 3800
 $Comp
-L GS3 J2
+L conn:GS3 J2
 U 1 1 5CA986BE
 P 8900 3600
@@
 $EndComp
 $Comp
-L MAX3378E U1
+L Libreria_SCH_mia1:MAX3378E U1
 U 1 1 5CAA29BD
 P 4200 3700
@@
 	5550 4050 5100 4050
 $Comp
-L CONN_01X06 J1
+L conn:CONN_01X06 J1
 U 1 1 5CAA3068
 P 1900 3150
@@
 	2100 3400 2100 3500
 $Comp
-L GND #PWR010
+L power:GND #PWR010
 U 1 1 5CAA33BE
 P 2100 3500
@@
 $EndComp
 $Comp
-L +5V #PWR011
+L power:+5V #PWR011
 U 1 1 5CAA3401
 P 5100 2550
@@
 $EndComp
 $Comp
-L GND #PWR012
+L power:GND #PWR012
 U 1 1 5CAA3425
 P 3300 4900
@@
 SS
 $Comp
-L +3.3V #PWR013
+L power:+3.3V #PWR013
 U 1 1 5CAA3727
 P 3350 2550
@@
 NoConn ~ 8250 3200
 $Comp
-L R R4
+L Device:R R4
 U 1 1 5CAA398D
 P 9300 3600
@@
 $EndComp
 $Comp
-L R R3
+L Device:R R3
 U 1 1 5CAA39BA
-P 9400 2500
-F 0 "R3" V 9480 2500 50  0000 C CNN
-F 1 "47k" V 9400 2500 50  0000 C CNN
-F 2 "Resistors_SMD:R_0805" V 9330 2500 50  0001 C CNN
-F 3 "" H 9400 2500 50  0001 C CNN
-	1    9400 2500
+P 10200 2500
+F 0 "R3" V 10280 2500 50  0000 C CNN
+F 1 "47k" V 10200 2500 50  0000 C CNN
+F 2 "Resistors_SMD:R_0805" V 10130 2500 50  0001 C CNN
+F 3 "" H 10200 2500 50  0001 C CNN
+	1    10200 2500
 	-1   0    0    -1
 $EndComp
 Wire Wire Line
-	9800 2350 9800 3400
+	9800 2350 9800 2850
 Wire Wire Line
 	9500 3600 9450 3600
 Wire Wire Line
-	9400 2650 9400 2850
-Wire Wire Line
-	9400 2850 9800 2850
+	10200 2650 10200 2850
+Wire Wire Line
+	10200 2850 9800 2850
 Connection ~ 9800 2850
 Wire Wire Line
@@
 	2650 2900 2100 2900
 Wire Wire Line
-	9400 2350 9400 2050
-Connection ~ 9400 2050
-Wire Wire Line
 	10000 2050 10200 2050
 Wire Wire Line
-	10200 2050 10200 1900
-$Comp
-L +5V #PWR014
+	10200 1900 10200 2050
+$Comp
+L power:+5V #PWR014
 U 1 1 5CAA3C5C
 P 10200 1900
@@
 $EndComp
 $Comp
-L GND #PWR015
+L power:GND #PWR015
 U 1 1 5CAA3CDC
 P 9800 3950
@@
 	6050 3400 6500 3400
 $Comp
-L R R1
+L Device:R R1
 U 1 1 5CAA46BA
 P 5700 4400
@@
 $EndComp
 $Comp
-L R R2
+L Device:R R2
 U 1 1 5CAA472A
 P 5700 5000
@@
 $EndComp
 Wire Wire Line
-	5700 4550 5700 4850
+	5700 4550 5700 4750
 Wire Wire Line
 	5100 4750 5700 4750
 Connection ~ 5700 4750
 $Comp
-L GND #PWR016
+L power:GND #PWR016
 U 1 1 5CAA4854
 P 5700 5200
@@
 SS
 $Comp
-L Q_NPN_BEC Q2
+L Device:Q_NPN_BEC Q2
 U 1 1 5CAA5338
 P 9700 3600
@@
 $EndComp
 $Comp
-L Q_PMOS_GDS Q1
+L Device:Q_PMOS_GDS Q1
 U 1 1 5CAA5695
 P 9800 2150
-F 0 "Q1" H 10000 2200 50  0000 L CNN
-F 1 "BSP315PH6327XTSA1" H 10000 2100 50  0000 L CNN
+F 0 "Q1" V 9750 2300 50  0000 L CNN
+F 1 "BSP315PH6327XTSA1" V 10050 1900 50  0000 L CNN
 F 2 "TO_SOT_Packages_SMD:SOT-223-3_TabPin2" H 10000 2250 50  0001 C CNN
 F 3 "" H 9800 2150 50  0001 C CNN
@@
 Text GLabel 8300 3600 2    60   Input ~ 0
 D6
+Connection ~ 10200 2050
+Wire Wire Line
+	9800 2850 9800 3400
+Wire Wire Line
+	5700 4750 5700 4850
+Wire Wire Line
+	10200 2050 10200 2350
 $EndSCHEMATC
