File: kicad/stima_v3/Microduino_RTC_DE/Microduino_RTC_DE.sch (KiCad schematic (older format))
At the start: 15 parts, among them P1 CONN_1x27, U1 PCF8563, Y1 32,762 kHz

Commit message: reapload kicad scheme
Parts:
- C1: symbol C_Small -> Device:C_Small
- C2: symbol CP -> Device:CP
- CV1: symbol C_Variable -> Device:C_Variable
- D1: symbol D_Schottky -> Device:D_Schottky
- D2: symbol D_Zener -> Device:D_Zener
- GS1, GS2: symbol GS3 -> conn:GS3
- GS3: symbol GS4 -> Libreria_SCH_mia:GS4
- P1: symbol CONN_1x27 -> Libreria_SCH_mia:CONN_1x27
- R1, R2, R3, R4: symbol R -> Device:R
- U1: symbol PCF8563 -> philips:PCF8563
- Y1: symbol Crystal -> Device:Crystal
Connections:
- wire segments 62 -> 78
- no-connect marks 21 -> 19
Changed lines of the file:
@@
-EESchema Schematic File Version 2
-LIBS:Libreria_SCH_mia
-LIBS:power
-LIBS:device
-LIBS:transistors
-LIBS:conn
-LIBS:linear
-LIBS:regul
-LIBS:74xx
-LIBS:cmos4000
-LIBS:adc-dac
-LIBS:memory
-LIBS:xilinx
-LIBS:microcontrollers
-LIBS:dsp
-LIBS:microchip
-LIBS:analog_switches
-LIBS:motorola
-LIBS:texas
-LIBS:intel
-LIBS:audio
-LIBS:interface
-LIBS:digital-audio
-LIBS:philips
-LIBS:display
-LIBS:cypress
-LIBS:siliconi
-LIBS:opto
-LIBS:atmel
-LIBS:contrib
-LIBS:valves
-LIBS:Microduino_RTC_DE-cache
-EELAYER 25 0
+EESchema Schematic File Version 4
+EELAYER 30 0
 EELAYER END
 $Descr A4 11693 8268
@@
 Sheet 1 1
 Title "Microduino RTC DE"
-Date "11 ottobre 2017"
+Date "24 dicembre 2017"
 Rev "0.1"
 Comp ""
@@
 $EndDescr
 $Comp
-L PCF8563 U1
+L philips:PCF8563 U1
 U 1 1 58B7F974
 P 3400 3800
@@
 $EndComp
 $Comp
-L Crystal Y1
+L Device:Crystal Y1
 U 1 1 58B7FA73
 P 2800 3800
@@
 $EndComp
 $Comp
-L C_Variable CV1
+L Device:C_Variable CV1
 U 1 1 58B7FAE6
 P 2800 3250
@@
 $EndComp
 $Comp
-L C_Small C1
+L Device:C_Small C1
 U 1 1 58B7FB48
 P 3800 3100
@@
 $EndComp
 $Comp
-L GND #PWR01
+L power:GND #PWR01
 U 1 1 58B7FC81
 P 3400 4400
@@
 $EndComp
 $Comp
-L R R1
+L Device:R R1
 U 1 1 58C44D2B
 P 4750 3200
@@
 $EndComp
 $Comp
-L R R2
+L Device:R R2
 U 1 1 58C44D52
 P 5000 3200
@@
 $EndComp
 $Comp
-L GND #PWR02
+L power:GND #PWR02
 U 1 1 58B7FE98
 P 3800 3250
@@
 $EndComp
 $Comp
-L CP C2
+L Device:CP C2
 U 1 1 58C58191
 P 2150 3650
@@
 $EndComp
 $Comp
-L D_Schottky D1
+L Device:D_Schottky D1
 U 1 1 58C5822F
 P 4500 2900
@@
 NoConn ~ 10150 4100
 $Comp
-L GND #PWR03
+L power:GND #PWR03
 U 1 1 58D4FFFC
 P 9800 4350
@@
 $EndComp
 $Comp
-L +5V #PWR04
+L power:+5V #PWR04
 U 1 1 58D50BEE
 P 7750 4200
@@
 $EndComp
 $Comp
-L +3.3V #PWR05
+L power:+3.3V #PWR05
 U 1 1 58D50CA7
 P 7950 4100
@@
 D13
 $Comp
-L +5V #PWR06
+L power:+5V #PWR06
 U 1 1 58D512B2
 P 6550 2800
@@
 $EndComp
 $Comp
-L +3.3V #PWR07
+L power:+3.3V #PWR07
 U 1 1 58D512DE
 P 6550 3000
@@
 A7
 Wire Wire Line
-	3400 4200 3400 4400
+	3400 4200 3400 4350
 Wire Wire Line
 	3000 3600 2800 3600
@@
 	3800 3200 3800 3250
 Wire Wire Line
-	3800 3600 5300 3600
-Wire Wire Line
-	3800 3700 5300 3700
+	3800 3600 4750 3600
+Wire Wire Line
+	3800 3700 5000 3700
 Wire Wire Line
 	5000 2900 5000 3050
@@
 Connection ~ 5000 3700
 Wire Wire Line
-	1500 2900 3950 2900
-Wire Wire Line
-	4650 2900 6150 2900
+	1500 2900 2150 2900
+Wire Wire Line
+	4650 2900 4750 2900
 Wire Wire Line
 	2800 2900 2800 3100
 Connection ~ 3400 2900
 Wire Wire Line
-	2800 3400 2800 3650
+	2800 3400 2800 3600
 Wire Wire Line
 	2800 4000 2800 3950
@@
 	2150 3800 2150 4350
 Wire Wire Line
-	1500 4350 3400 4350
+	1500 4350 2150 4350
 Connection ~ 3400 4350
 Connection ~ 5000 2900
@@
 Wire Wire Line
 	8800 2850 8800 3100
-NoConn ~ 9300 2850
-NoConn ~ 9200 2850
 Text Label 5300 3600 2    60   ~ 0
 SCL
@@
 INT
 $Comp
-L PWR_FLAG #FLG08
-U 1 1 58D52798
-P 2150 4350
-F 0 "#FLG08" H 2150 4445 50  0001 C CNN
-F 1 "PWR_FLAG" H 2150 4530 50  0000 C CNN
-F 2 "" H 2150 4350 50  0000 C CNN
-F 3 "" H 2150 4350 50  0000 C CNN
-	1    2150 4350
-	-1   0    0    1
-$EndComp
-$Comp
-L PWR_FLAG #FLG09
+L power:PWR_FLAG #FLG08
 U 1 1 58D527C4
 P 2150 2900
-F 0 "#FLG09" H 2150 2995 50  0001 C CNN
+F 0 "#FLG08" H 2150 2995 50  0001 C CNN
 F 1 "PWR_FLAG" H 2150 3080 50  0000 C CNN
 F 2 "" H 2150 2900 50  0000 C CNN
@@
 	10150 4000 9800 4000
 $Comp
-L GS3 GS1
+L conn:GS3 GS1
 U 1 1 58D9FACF
 P 6300 2900
@@
 $EndComp
 $Comp
-L R R3
+L Device:R R3
 U 1 1 58DA426D
 P 5700 3450
@@
 	6550 3900 6450 3900
 $Comp
-L GS3 GS2
+L conn:GS3 GS2
 U 1 1 58D9FB5B
 P 5150 4000
@@
 $EndComp
 Wire Wire Line
-	5300 4000 6150 4000
+	5300 4000 5700 4000
 Wire Wire Line
 	5000 3900 3800 3900
@@
 	4400 4100 5000 4100
 $Comp
-L D_Zener D2
+L Device:D_Zener D2
 U 1 1 58E73E8C
 P 1500 3650
@@
 $EndComp
 $Comp
-L R R4
+L Device:R R4
 U 1 1 58E74C0B
 P 4100 2900
@@
 UPIN 27
 $Comp
-L CONN_1x27 P1
+L Libreria_SCH_mia:CONN_1x27 P1
 U 1 1 58E8E495
 P 8600 4200
@@
 DigitEco s.r.l.
 $Comp
-L GS4 GS3
+L Libreria_SCH_mia:GS4 GS3
 U 1 1 59DEFC44
 P 6300 4000
@@
 Wire Wire Line
 	6450 4200 6550 4200
+$Comp
+L power:+3.3V #PWR09
+U 1 1 5A3F82F5
+P 8550 5400
+F 0 "#PWR09" H 8550 5250 50  0001 C CNN
+F 1 "+3.3V" H 8550 5540 50  0000 C CNN
+F 2 "" H 8550 5400 50  0001 C CNN
+F 3 "" H 8550 5400 50  0001 C CNN
+	1    8550 5400
+	1    0    0    -1
+$EndComp
+$Comp
+L power:+5V #PWR010
+U 1 1 5A3F8327
+P 9100 5400
+F 0 "#PWR010" H 9100 5250 50  0001 C CNN
+F 1 "+5V" H 9100 5540 50  0000 C CNN
+F 2 "" H 9100 5400 50  0001 C CNN
+F 3 "" H 9100 5400 50  0001 C CNN
+	1    9100 5400
+	1    0    0    -1
+$EndComp
+$Comp
+L power:GND #PWR011
+U 1 1 5A3F8359
+P 9650 5600
+F 0 "#PWR011" H 9650 5350 50  0001 C CNN
+F 1 "GND" H 9650 5450 50  0000 C CNN
+F 2 "" H 9650 5600 50  0001 C CNN
+F 3 "" H 9650 5600 50  0001 C CNN
+	1    9650 5600
+	1    0    0    -1
+$EndComp
+$Comp
+L power:PWR_FLAG #FLG012
+U 1 1 5A3F838B
+P 9650 5400
+F 0 "#FLG012" H 9650 5475 50  0001 C CNN
+F 1 "PWR_FLAG" H 9650 5550 50  0000 C CNN
+F 2 "" H 9650 5400 50  0001 C CNN
+F 3 "" H 9650 5400 50  0001 C CNN
+	1    9650 5400
+	1    0    0    -1
+$EndComp
+$Comp
+L power:PWR_FLAG #FLG013
+U 1 1 5A3F83BD
+P 9100 5600
+F 0 "#FLG013" H 9100 5675 50  0001 C CNN
+F 1 "PWR_FLAG" H 9100 5750 50  0000 C CNN
+F 2 "" H 9100 5600 50  0001 C CNN
+F 3 "" H 9100 5600 50  0001 C CNN
+	1    9100 5600
+	-1   0    0    1
+$EndComp
+$Comp
+L power:PWR_FLAG #FLG014
+U 1 1 5A3F83EF
+P 8550 5600
+F 0 "#FLG014" H 8550 5675 50  0001 C CNN
+F 1 "PWR_FLAG" H 8550 5750 50  0000 C CNN
+F 2 "" H 8550 5600 50  0001 C CNN
+F 3 "" H 8550 5600 50  0001 C CNN
+	1    8550 5600
+	-1   0    0    1
+$EndComp
+Wire Wire Line
+	8550 5400 8550 5600
+Wire Wire Line
+	9100 5400 9100 5600
+Wire Wire Line
+	9650 5400 9650 5600
+Wire Wire Line
+	3800 2900 3950 2900
+Wire Wire Line
+	4750 2900 5000 2900
+Wire Wire Line
+	4750 3600 5300 3600
+Wire Wire Line
+	5000 3700 5300 3700
+Wire Wire Line
+	3400 2900 3800 2900
+Wire Wire Line
+	2800 2900 3400 2900
+Wire Wire Line
+	3400 4350 3400 4400
+Wire Wire Line
+	5000 2900 5700 2900
+Wire Wire Line
+	2800 3600 2800 3650
+Wire Wire Line
+	5700 2900 6150 2900
+Wire Wire Line
+	5700 4000 6150 4000
+Wire Wire Line
+	2150 2900 2800 2900
+Wire Wire Line
+	2150 4350 3400 4350
 $EndSCHEMATC
