File: kicad/stima_v3/Microduino_SD_DE/Microduino_SD_DE.kicad_pcb (KiCad board)
At the start: 2 copper layers, 25.5 x 27.9 mm, 6 parts, among them P1 CONN_1x27, U1 4050

Commit message: reapload kicad scheme
Connections:
- D1 pad 1: Net-(CARD1-Pad2) -> GND
- R1 pad 2: Net-(R1-Pad2) -> /D4
- U1 pad 10: Net-(R1-Pad2) -> Net-(U1-Pad10)
- U1 pad 9: /CLK -> Net-(U1-Pad9)
Routing:
- net /D4: track 0.00 -> 19.1 mm, vias 0 -> 1
- net Net-(CARD1-Pad2): track 23.2 -> 13.4 mm
- net GND: track 71.8 -> 80.4 mm
- net Net-(R1-Pad2): track 5.62 -> 0.00 mm
- net /CLK: track 24.0 -> 18.9 mm
Changed lines of the file:
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@@
 (kicad_pcb (version 4) (host pcbnew 4.0.6)
   (general
-    (links 23)
+    (links 22)
     (no_connects 0)
     (area 138.634399 62.662999 164.311401 90.753001)
     (thickness 1.6)
     (drawings 54)
-    (tracks 95)
+    (tracks 100)
     (zones 0)
     (modules 6)
-    (nets 37)
+    (nets 38)
   )
   (page A4)
   (title_block
     (title "Microduino SD DE")
-    (date "30 luglio 2017")
-    (rev 0.0)
+    (date "06 aprile 2019")
+    (rev 0.1)
   )
   (layers
@@
   )
   (setup
-    (last_trace_width 0.4)
+    (last_trace_width 0.25)
     (user_trace_width 0.4)
     (user_trace_width 0.5)
@@
   (net 31 /D2)
   (net 32 /D3)
-  (net 33 "Net-(R1-Pad2)")
-  (net 34 "Net-(U1-Pad12)")
-  (net 35 "Net-(U1-Pad15)")
-  (net 36 "Net-(CARD1-Pad8)")
+  (net 33 "Net-(U1-Pad12)")
+  (net 34 "Net-(U1-Pad15)")
+  (net 35 "Net-(CARD1-Pad8)")
+  (net 36 "Net-(U1-Pad9)")
+  (net 37 "Net-(U1-Pad10)")
   (net_class Default "Questo è il gruppo di collegamenti predefinito"
     (clearance 0.2)
@@
     (add_net "Net-(CARD1-Pad8)")
     (add_net "Net-(D1-Pad2)")
-    (add_net "Net-(R1-Pad2)")
+    (add_net "Net-(U1-Pad10)")
     (add_net "Net-(U1-Pad12)")
     (add_net "Net-(U1-Pad15)")
+    (add_net "Net-(U1-Pad9)")
   )
   (module Libreria_PCB_mia:Upin_27 (layer B.Cu)
@@
     (pad 27 thru_hole circle (at 20.32 0 180) (size 2.1 2.1) (drill 1.5) (layers *.Cu *.Mask)
       (net 18 GND))
-    (model ${KISYS3DMOD}/Socket_Strips.3dshapes/Socket_Strip_Straight_1x09_Pitch2.54mm.wrl
-      (at (xyz 0 -0.4 0))
-      (scale (xyz 1 1 1))
-      (rotate (xyz 0 0 270))
-    )
   )
   (module Capacitors_SMD:C_0805 (layer F.Cu)
@@
       (net 18 GND))
     (pad 8 smd rect (at 4.5 -2.7 180) (size 0.8 1.5) (layers F.Cu F.Paste F.Mask)
-      (net 36 "Net-(CARD1-Pad8)"))
+      (net 35 "Net-(CARD1-Pad8)"))
     (pad 7 smd rect (at 3.4 -2.7 180) (size 0.8 1.5) (layers F.Cu F.Paste F.Mask)
       (net 20 /DO))
@@
       (net 25 "Net-(D1-Pad2)"))
     (pad 1 smd rect (at -1.1 0 270) (size 1.2 1.2) (layers F.Cu F.Paste F.Mask)
-      (net 23 "Net-(CARD1-Pad2)"))
+      (net 18 GND))
     (model ${KISYS3DMOD}/LEDs.3dshapes/LED_0805.wrl
       (at (xyz 0 0 0))
@@
       (net 25 "Net-(D1-Pad2)"))
     (pad 2 smd rect (at 0.95 0 90) (size 0.7 1.3) (layers F.Cu F.Paste F.Mask)
-      (net 33 "Net-(R1-Pad2)"))
+      (net 14 /D4))
     (model ${KISYS3DMOD}/Resistors_SMD.3dshapes/R_0805.wrl
       (at (xyz 0 0 0))
@@
       (net 18 GND))
     (pad 9 smd rect (at 2.95 2.275 90) (size 1.5 0.45) (layers F.Cu F.Paste F.Mask)
-      (net 26 /CLK))
+      (net 36 "Net-(U1-Pad9)"))
     (pad 10 smd rect (at 2.95 1.625 90) (size 1.5 0.45) (layers F.Cu F.Paste F.Mask)
-      (net 33 "Net-(R1-Pad2)"))
+      (net 37 "Net-(U1-Pad10)"))
     (pad 11 smd rect (at 2.95 0.975 90) (size 1.5 0.45) (layers F.Cu F.Paste F.Mask)
       (net 18 GND))
     (pad 12 smd rect (at 2.95 0.325 90) (size 1.5 0.45) (layers F.Cu F.Paste F.Mask)
-      (net 34 "Net-(U1-Pad12)"))
+      (net 33 "Net-(U1-Pad12)"))
     (pad 13 smd rect (at 2.95 -0.325 90) (size 1.5 0.45) (layers F.Cu F.Paste F.Mask))
     (pad 14 smd rect (at 2.95 -0.975 90) (size 1.5 0.45) (layers F.Cu F.Paste F.Mask)
       (net 18 GND))
     (pad 15 smd rect (at 2.95 -1.625 90) (size 1.5 0.45) (layers F.Cu F.Paste F.Mask)
-      (net 35 "Net-(U1-Pad15)"))
+      (net 34 "Net-(U1-Pad15)"))
     (pad 16 smd rect (at 2.95 -2.275 90) (size 1.5 0.45) (layers F.Cu F.Paste F.Mask))
     (model ${KISYS3DMOD}/Housings_SSOP.3dshapes/TSSOP-16_4.4x5mm_Pitch0.65mm.wrl
@@
   (via (at 151.301 81.215) (size 0.6) (drill 0.4) (layers F.Cu B.Cu) (net 2))
   (segment (start 151.301 81.215) (end 151.311 81.225) (width 0.4) (layer F.Cu) (net 2))
+  (segment (start 154.341 70.775) (end 152.563 70.775) (width 0.4) (layer F.Cu) (net 14))
+  (segment (start 143.1036 78.0034) (end 141.2494 78.0034) (width 0.4) (layer B.Cu) (net 14))
+  (segment (start 143.891 77.216) (end 143.1036 78.0034) (width 0.4) (layer B.Cu) (net 14))
+  (segment (start 143.891 72.136) (end 143.891 77.216) (width 0.4) (layer B.Cu) (net 14))
+  (segment (start 145.288 70.739) (end 143.891 72.136) (width 0.4) (layer B.Cu) (net 14))
+  (segment (start 150.876 70.739) (end 145.288 70.739) (width 0.4) (layer B.Cu) (net 14))
+  (segment (start 152.527 70.739) (end 150.876 70.739) (width 0.4) (layer B.Cu) (net 14))
+  (via (at 152.527 70.739) (size 0.6) (drill 0.4) (layers F.Cu B.Cu) (net 14))
+  (segment (start 152.563 70.775) (end 152.527 70.739) (width 0.4) (layer F.Cu) (net 14))
+  (segment (start 151.026 74.555) (end 151.026 73.429) (width 0.4) (layer F.Cu) (net 18))
+  (segment (start 152.541 73.735) (end 156.861 73.735) (width 0.4) (layer F.Cu) (net 18))
+  (segment (start 156.861 73.735) (end 157.801 72.795) (width 0.4) (layer F.Cu) (net 18))
+  (segment (start 152.602 73.735) (end 152.541 73.735) (width 0.4) (layer F.Cu) (net 18))
+  (segment (start 152.146 73.279) (end 152.602 73.735) (width 0.4) (layer F.Cu) (net 18))
+  (segment (start 151.176 73.279) (end 152.146 73.279) (width 0.4) (layer F.Cu) (net 18))
+  (segment (start 151.026 73.429) (end 151.176 73.279) (width 0.4) (layer F.Cu) (net 18))
   (via (at 156.361 80.655) (size 0.6) (drill 0.4) (layers F.Cu B.Cu) (net 18))
   (segment (start 144.536 80.655) (end 146.361 80.655) (width 0.4) (layer F.Cu) (net 18))
@@
   (segment (start 155.601 77.915) (end 158.801 74.715) (width 0.4) (layer B.Cu) (net 20))
   (segment (start 161.5694 70.3834) (end 159.4426 70.3834) (width 0.4) (layer B.Cu) (net 20))
-  (segment (start 148.011 84.655) (end 148.011 86.355) (width 0.4) (layer F.Cu) (net 20) (status 800000))
+  (segment (start 148.011 84.655) (end 148.011 86.355) (width 0.4) (layer F.Cu) (net 20))
   (via (at 148.011 84.655) (size 0.6) (drill 0.4) (layers F.Cu B.Cu) (net 20))
   (segment (start 148.011 84.665) (end 148.011 84.655) (width 0.4) (layer B.Cu) (net 20))
@@
   (segment (start 152.411 80.745) (end 152.411 86.355) (width 0.4) (layer F.Cu) (net 22))
   (segment (start 148.426 76.76) (end 152.411 80.745) (width 0.4) (layer F.Cu) (net 22))
-  (segment (start 149.726 74.555) (end 149.726 73.48853) (width 0.4) (layer F.Cu) (net 23))
-  (segment (start 156.861 73.735) (end 157.801 72.795) (width 0.4) (layer F.Cu) (net 23))
-  (segment (start 152.541 73.735) (end 156.861 73.735) (width 0.4) (layer F.Cu) (net 23))
-  (segment (start 152.001 73.195) (end 152.541 73.735) (width 0.4) (layer F.Cu) (net 23))
-  (segment (start 150.01953 73.195) (end 152.001 73.195) (width 0.4) (layer F.Cu) (net 23))
-  (segment (start 149.726 73.48853) (end 150.01953 73.195) (width 0.4) (layer F.Cu) (net 23))
   (segment (start 149.726 74.555) (end 149.726 76.47) (width 0.4) (layer F.Cu) (net 23))
   (segment (start 153.511 80.255) (end 153.511 86.355) (width 0.4) (layer F.Cu) (net 23))
@@
   (segment (start 154.341 72.675) (end 155.721 72.675) (width 0.4) (layer F.Cu) (net 25))
   (segment (start 155.721 72.675) (end 157.801 70.595) (width 0.4) (layer F.Cu) (net 25))
-  (segment (start 156.161 68.655) (end 156.161 71.105) (width 0.4) (layer F.Cu) (net 26))
+  (segment (start 156.161 71.105) (end 156.161 68.629) (width 0.4) (layer F.Cu) (net 26))
+  (segment (start 155.551 71.715) (end 156.161 71.105) (width 0.4) (layer F.Cu) (net 26))
+  (segment (start 147.776 74.555) (end 147.776 73.09) (width 0.4) (layer F.Cu) (net 26))
+  (segment (start 149.151 71.715) (end 155.551 71.715) (width 0.4) (layer F.Cu) (net 26))
   (segment (start 147.776 73.09) (end 149.151 71.715) (width 0.4) (layer F.Cu) (net 26))
-  (segment (start 149.151 71.715) (end 155.551 71.715) (width 0.4) (layer F.Cu) (net 26))
-  (segment (start 155.551 71.715) (end 156.161 71.105) (width 0.4) (layer F.Cu) (net 26))
-  (segment (start 147.776 73.09) (end 147.776 74.555) (width 0.4) (layer F.Cu) (net 26))
-  (segment (start 151.026 68.655) (end 156.161 68.655) (width 0.4) (layer F.Cu) (net 26))
-  (segment (start 156.161 68.655) (end 157.891 68.655) (width 0.4) (layer F.Cu) (net 26))
-  (segment (start 158.7026 67.8434) (end 161.5694 67.8434) (width 0.4) (layer F.Cu) (net 26))
-  (segment (start 157.891 68.655) (end 158.7026 67.8434) (width 0.4) (layer F.Cu) (net 26))
+  (segment (start 156.9466 67.8434) (end 161.5694 67.8434) (width 0.4) (layer F.Cu) (net 26))
+  (segment (start 156.161 68.629) (end 156.9466 67.8434) (width 0.4) (layer F.Cu) (net 26))
   (segment (start 160.5326 72.9234) (end 161.5694 72.9234) (width 0.4) (layer F.Cu) (net 27))
   (segment (start 158.751 74.705) (end 160.5326 72.9234) (width 0.4) (layer F.Cu) (net 27))
@@
   (segment (start 154.591 80.105) (end 154.591 81.805) (width 0.4) (layer F.Cu) (net 28))
   (segment (start 150.376 75.89) (end 154.591 80.105) (width 0.4) (layer F.Cu) (net 28))
-  (segment (start 150.376 68.655) (end 150.376 69.98) (width 0.4) (layer F.Cu) (net 33))
-  (segment (start 151.171 70.775) (end 154.341 70.775) (width 0.4) (layer F.Cu) (net 33))
-  (segment (start 150.376 69.98) (end 151.171 70.775) (width 0.4) (layer F.Cu) (net 33))
 )
