File: kicad/stima_v3/Microduino_SD_DE/Microduino_SD_DE.sch (KiCad schematic (older format))
At the start: 6 parts, among them P1 CONN_1x27, U1 4050

Commit message: reapload kicad scheme
Parts:
- C1: symbol C -> Device:C
- CARD1: symbol Micro_SD_Card -> conn:Micro_SD_Card
- D1: symbol LED_ALT -> Device:LED_ALT
- P1: symbol CONN_1x27 -> Microduino_SD_DE-rescue:CONN_1x27-Libreria_SCH_mia
- R1: symbol R -> Device:R
- U1: symbol 4050 -> cmos4000:4050
Connections:
- wire segments 60 -> 58
- no-connect marks 24 -> 25
