File: kicad/stima_v3/Microduino_SUPPORTO_DE/Microduino_Supporto_DE.sch (KiCad schematic (older format))
At the start: 1 part, among them P1 CONN_1x27

Commit message: reapload kicad scheme
Other:
- moved on the sheet: P1
