File: kicad/stima_v3/Microduino_UART/Microduino_UART.kicad_pcb (KiCad board)
At the start: 2 copper layers, 25.5 x 27.9 mm, 18 parts, among them J1 Conn_01x05, P1 CONN_1x27, Q1 Q1, Q2 Q2, U1 MAX3232

Commit message: reapload kicad scheme
Parts:
- added GS2: GS3, Connectors:GS3, B.Cu at (157.9, 82.5)
- Q1: value Q1 -> BSP315PH6327XTSA1
- Q2: value Q2 -> BC847B
Changed lines of the file:
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@@
-(kicad_pcb (version 20171130) (host pcbnew 5.1.5+dfsg1-2build2)
+(kicad_pcb (version 20171130) (host pcbnew "(5.1.5)-3")
   (general
     (thickness 1.6)
@@
     (tracks 190)
     (zones 0)
-    (modules 18)
+    (modules 19)
     (nets 46)
   )
@@
       (effects (font (size 1 1) (thickness 0.15)))
     )
-    (fp_text value Q1 (at 0 4.5) (layer F.Fab)
+    (fp_text value BSP315PH6327XTSA1 (at 0 4.5) (layer F.Fab)
       (effects (font (size 1 1) (thickness 0.15)))
     )
@@
       (effects (font (size 0.6444 0.6444) (thickness 0.1246)) (justify mirror))
     )
-    (fp_text value Q2 (at 0 -2.5) (layer B.Fab)
+    (fp_text value BC847B (at 0 -2.5) (layer B.Fab)
       (effects (font (size 1 1) (thickness 0.15)) (justify mirror))
     )
@@
     )
   )
+  (module Connectors:GS3 (layer B.Cu)
+    (at 157.9499 82.4738)
+    (descr "3-pin solder bridge")
+    (tags "solder bridge")
+    (attr smd)
+    (fp_text reference GS2 (at -1.7 0 270) (layer B.SilkS)
+      (effects (font (size 0.6444 0.6444) (thickness 0.0992)) (justify mirror))
+    )
+    (fp_text value GS3 (at 1.8 0 270) (layer B.Fab)
+      (effects (font (size 1 1) (thickness 0.15)) (justify mirror))
+    )
+    (fp_line (start -1.15 2.15) (end 1.15 2.15) (layer B.CrtYd) (width 0.05))
+    (fp_line (start 1.15 2.15) (end 1.15 -2.15) (layer B.CrtYd) (width 0.05))
+    (fp_line (start 1.15 -2.15) (end -1.15 -2.15) (layer B.CrtYd) (width 0.05))
+    (fp_line (start -1.15 -2.15) (end -1.15 2.15) (layer B.CrtYd) (width 0.05))
+    (fp_line (start -0.89 1.91) (end -0.89 -1.91) (layer B.SilkS) (width 0.12))
+    (fp_line (start -0.89 -1.91) (end 0.89 -1.91) (layer B.SilkS) (width 0.12))
+    (fp_line (start 0.89 -1.91) (end 0.89 1.91) (layer B.SilkS) (width 0.12))
+    (fp_line (start -0.89 1.91) (end 0.89 1.91) (layer B.SilkS) (width 0.12))
+    (pad 1 smd rect (at 0 1.27) (size 1.27 0.97) (layers B.Cu B.Paste B.Mask)
+      (net 1 +5V))
+    (pad 2 smd rect (at 0 0) (size 1.27 0.97) (layers B.Cu B.Paste B.Mask)
+      (net 43 "Net-(C1-Pad1)"))
+    (pad 3 smd rect (at 0 -1.27) (size 1.27 0.97) (layers B.Cu B.Paste B.Mask)
+      (net 2 +3V3))
+  )
   (module Capacitors_Tantalum_SMD:CP_Tantalum_Case-B_EIA-3528-21_Reflow (layer B.Cu)
