File: kicad/stima_v3/Microduino_UART/Microduino_UART.sch (KiCad schematic (older format))
At the start: 19 parts, among them J1 Conn_01x05, P1 CONN_1x27, Q1 Q1, Q2 Q2, U1 MAX3232

Commit message: reapload kicad scheme
Parts:
- removed JP3: SolderJumper_3_Open, Connectors:GS3, symbol Jumper:SolderJumper_3_Open
- added GS2: GS3, Connectors:GS3, symbol conn:GS3
- C1, C2, C3, C4, C5, C6, C7: Codice (none) -> C1206C104K5RACTU; Codice Mouser (none) -> 80-C1206C104K5R; Codice RS (none) -> 391-214
- Q1: value Q1 -> BSP315PH6327XTSA1; Codice (none) -> BSP315PH6327XTSA1; Codice Mouser (none) -> 726-BSP315PH6327XTSA; Codice RS (none) -> 826-9238
- Q2: value Q2 -> BC847B; Codice (none) -> BC847B,215; Codice Mouser (none) -> 771-BC847B-T/R; Codice RS (none) -> 436-7947
- R1: Codice (none) -> CRCW120647K0FKEA; Codice Mouser (none) -> 71-CRCW1206-47K-E3; Codice RS (none) -> 679-2156
- R2: Codice (none) -> CRCW12064K70FKEA; Codice Mouser (none) -> 71-CRCW1206-4.7K-E3; Codice RS (none) -> 679-2184
Connections:
- net +3V3: now also GS2.3 (G3)
- net +5V: now also GS2.1 (G1)
- net at C1.1, U1.16 (VCC): now also GS2.2 (G2)
Changed lines of the file:
@@
 F 2 "Capacitor_SMD:C_0805_2012Metric" H 3988 2875 50  0001 C CNN
 F 3 "" H 3950 3025 50  0000 C CNN
-F 4 "" H 3950 3025 50  0001 C CNN "Codice"
-F 5 "m" H 3950 3025 50  0001 C CNN "Campo4"
+F 4 "C1206C104K5RACTU" H 3950 3025 50  0001 C CNN "Codice"
+F 5 "391-214" H 3950 3025 50  0001 C CNN "Codice RS"
+F 6 "m" H 3950 3025 50  0001 C CNN "Campo4"
+F 7 "80-C1206C104K5R" H 3950 3025 50  0001 C CNN "Codice Mouser"
 	1    3950 3025
 	-1   0    0    -1
@@
 F 2 "Capacitor_SMD:C_0805_2012Metric" H 5388 3575 50  0001 C CNN
 F 3 "" H 5350 3725 50  0000 C CNN
-F 4 "" H 5350 3725 50  0001 C CNN "Codice"
-F 5 "m" H 5350 3725 50  0001 C CNN "Campo4"
+F 4 "C1206C104K5RACTU" H 5350 3725 50  0001 C CNN "Codice"
+F 5 "391-214" H 5350 3725 50  0001 C CNN "Codice RS"
+F 6 "m" H 5350 3725 50  0001 C CNN "Campo4"
+F 7 "80-C1206C104K5R" H 5350 3725 50  0001 C CNN "Codice Mouser"
 	1    5350 3725
 	1    0    0    -1
@@
 F 2 "Capacitor_SMD:C_0805_2012Metric" H 3388 3575 50  0001 C CNN
 F 3 "" H 3350 3725 50  0000 C CNN
-F 4 "" H 3350 3725 50  0001 C CNN "Codice"
-F 5 "m" H 3350 3725 50  0001 C CNN "Campo4"
+F 4 "C1206C104K5RACTU" H 3350 3725 50  0001 C CNN "Codice"
+F 5 "391-214" H 3350 3725 50  0001 C CNN "Codice RS"
+F 6 "m" H 3350 3725 50  0001 C CNN "Campo4"
+F 7 "80-C1206C104K5R" H 3350 3725 50  0001 C CNN "Codice Mouser"
 	1    3350 3725
 	-1   0    0    -1
@@
 F 2 "Capacitor_SMD:C_0805_2012Metric" H 3238 3925 50  0001 C CNN
 F 3 "" H 3200 4075 50  0000 C CNN
-F 4 "" H 3200 4075 50  0001 C CNN "Codice"
-F 5 "m" H 3200 4075 50  0001 C CNN "Campo4"
+F 4 "C1206C104K5RACTU" H 3200 4075 50  0001 C CNN "Codice"
+F 5 "391-214" H 3200 4075 50  0001 C CNN "Codice RS"
+F 6 "m" H 3200 4075 50  0001 C CNN "Campo4"
+F 7 "80-C1206C104K5R" H 3200 4075 50  0001 C CNN "Codice Mouser"
 	1    3200 4075
 	0    -1   1    0
@@
 F 2 "Capacitor_SMD:C_0805_2012Metric" H 3238 4225 50  0001 C CNN
 F 3 "" H 3200 4375 50  0000 C CNN
-F 4 "" H 3200 4375 50  0001 C CNN "Codice"
-F 5 "m" H 3200 4375 50  0001 C CNN "Campo4"
+F 4 "C1206C104K5RACTU" H 3200 4375 50  0001 C CNN "Codice"
+F 5 "391-214" H 3200 4375 50  0001 C CNN "Codice RS"
+F 6 "m" H 3200 4375 50  0001 C CNN "Campo4"
+F 7 "80-C1206C104K5R" H 3200 4375 50  0001 C CNN "Codice Mouser"
 	1    3200 4375
 	0    1    -1   0
@@
 	2900 4375 2900 4425
 Wire Wire Line
+	4350 2625 4350 2775
+Wire Wire Line
 	3950 2775 4350 2775
+Connection ~ 4350 2775
+Wire Wire Line
+	4350 2775 4350 3275
 Wire Wire Line
 	1900 4575 3550 4575
@@
 F 2 "Resistor_SMD:R_0805_2012Metric" V 7155 2675 50  0001 C CNN
 F 3 "" H 7225 2675 50  0001 C CNN
-F 4 "" H 7225 2675 50  0001 C CNN "Codice"
-F 5 "rs" H 7225 2675 50  0001 C CNN "Campo4"
+F 4 "CRCW12064K70FKEA" H 7225 2675 50  0001 C CNN "Codice"
+F 5 "679-2184" H 7225 2675 50  0001 C CNN "Codice RS"
+F 6 "rs" H 7225 2675 50  0001 C CNN "Campo4"
+F 7 "71-CRCW1206-4.7K-E3" H 7225 2675 50  0001 C CNN "Codice Mouser"
 	1    7225 2675
 	0    -1   -1   0
@@
 F 2 "Resistor_SMD:R_0805_2012Metric" V 7005 1925 50  0001 C CNN
 F 3 "" H 7075 1925 50  0001 C CNN
-F 4 "" H 7075 1925 50  0001 C CNN "Codice"
-F 5 "m" H 7075 1925 50  0001 C CNN "Campo4"
+F 4 "CRCW120647K0FKEA" H 7075 1925 50  0001 C CNN "Codice"
+F 5 "679-2156" H 7075 1925 50  0001 C CNN "Codice RS"
+F 6 "m" H 7075 1925 50  0001 C CNN "Campo4"
+F 7 "71-CRCW1206-47K-E3" H 7075 1925 50  0001 C CNN "Codice Mouser"
 	1    7075 1925
 	-1   0    0    -1
@@
 AR Path="/5FA30BCD" Ref="Q2"  Part="1"
 F 0 "Q2" H 6975 2725 50  0000 L CNN
-F 1 "Q2" H 6975 2625 50  0000 L CNN
+F 1 "BC847B" H 6975 2625 50  0000 L CNN
 F 2 "Package_TO_SOT_SMD:SOT-23" H 6975 2775 50  0001 C CNN
 F 3 "" H 6775 2675 50  0001 C CNN
-F 4 "" H 6775 2675 50  0001 C CNN "Codice"
-F 5 "m" H 6775 2675 50  0001 C CNN "Campo4"
+F 4 "BC847B,215" H 6775 2675 50  0001 C CNN "Codice"
+F 5 "436-7947" H 6775 2675 50  0001 C CNN "Codice RS"
+F 6 "m" H 6775 2675 50  0001 C CNN "Campo4"
+F 7 "771-BC847B-T/R" H 6775 2675 50  0001 C CNN "Codice Mouser"
 	1    6775 2675
 	-1   0    0    -1
@@
 AR Path="/5FA30BD7" Ref="Q1"  Part="1"
 F 0 "Q1" V 6625 1875 50  0000 L CNN
-F 1 "Q1" V 6925 1325 50  0000 L CNN
+F 1 "BSP315PH6327XTSA1" V 6925 1325 50  0000 L CNN
 F 2 "Package_TO_SOT_SMD:SOT-223-3_TabPin2" H 6875 1825 50  0001 C CNN
 F 3 "" H 6675 1725 50  0001 C CNN
-F 4 "" H 6675 1725 50  0001 C CNN "Codice"
-F 5 "m" H 6675 1725 50  0001 C CNN "Campo4"
+F 4 "BSP315PH6327XTSA1" H 6675 1725 50  0001 C CNN "Codice"
+F 5 "826-9238" H 6675 1725 50  0001 C CNN "Codice RS"
+F 6 "m" H 6675 1725 50  0001 C CNN "Campo4"
+F 7 "726-BSP315PH6327XTSA" H 6675 1725 50  0001 C CNN "Codice Mouser"
 	1    6675 1725
 	0    -1   -1   0
@@
 	10025 4200 9575 4200
 $Comp
+L power:+5V #PWR0110
+U 1 1 5FA1B659
+P 4250 2250
+F 0 "#PWR0110" H 4250 2100 50  0001 C CNN
+F 1 "+5V" H 4200 2425 50  0000 C CNN
+F 2 "" H 4250 2250 50  0001 C CNN
+F 3 "" H 4250 2250 50  0001 C CNN
+	1    4250 2250
+	1    0    0    -1
+$EndComp
+$Comp
 L power:+5V #PWR0111
 U 1 1 5FA1BBE0
@@
 Wire Wire Line
 	5675 4575 5150 4575
+$Comp
+L conn:GS3 GS2
+U 1 1 5FB43326
+P 4350 2475
+F 0 "GS2" V 4350 2287 50  0000 R CNN
+F 1 "GS3" V 4395 2287 50  0001 R CNN
+F 2 "Connectors:GS3" V 4438 2401 50  0001 C CNN
+F 3 "" H 4350 2475 50  0001 C CNN
+	1    4350 2475
+	0    -1   1    0
+$EndComp
+$Comp
+L power:+3.3V #PWR0117
+U 1 1 5FB43EC1
+P 4450 2250
+F 0 "#PWR0117" H 4450 2100 50  0001 C CNN
+F 1 "+3.3V" H 4500 2425 50  0000 C CNN
+F 2 "" H 4450 2250 50  0001 C CNN
+F 3 "" H 4450 2250 50  0001 C CNN
+	1    4450 2250
+	1    0    0    -1
+$EndComp
+Wire Wire Line
+	4250 2250 4250 2325
+Wire Wire Line
+	4450 2250 4450 2325
 $Comp
 L Device:C C?
@@
 F 2 "Capacitor_SMD:C_0805_2012Metric" H 2288 4975 50  0001 C CNN
 F 3 "" H 2250 5125 50  0000 C CNN
-F 4 "" H 2250 5125 50  0001 C CNN "Codice"
-F 5 "m" H 2250 5125 50  0001 C CNN "Campo4"
+F 4 "C1206C104K5RACTU" H 2250 5125 50  0001 C CNN "Codice"
+F 5 "391-214" H 2250 5125 50  0001 C CNN "Codice RS"
+F 6 "m" H 2250 5125 50  0001 C CNN "Campo4"
+F 7 "80-C1206C104K5R" H 2250 5125 50  0001 C CNN "Codice Mouser"
 	1    2250 5125
 	-1   0    0    -1
@@
 F 2 "Capacitor_SMD:C_0805_2012Metric" H 2538 4975 50  0001 C CNN
 F 3 "" H 2500 5125 50  0000 C CNN
-F 4 "" H 2500 5125 50  0001 C CNN "Codice"
-F 5 "m" H 2500 5125 50  0001 C CNN "Campo4"
+F 4 "C1206C104K5RACTU" H 2500 5125 50  0001 C CNN "Codice"
+F 5 "391-214" H 2500 5125 50  0001 C CNN "Codice RS"
+F 6 "m" H 2500 5125 50  0001 C CNN "Campo4"
+F 7 "80-C1206C104K5R" H 2500 5125 50  0001 C CNN "Codice Mouser"
 	1    2500 5125
 	1    0    0    -1
@@
 Wire Wire Line
 	2500 4850 2500 4975
-$Comp
-L power:+5V #PWR0110
-U 1 1 5FA1B659
-P 4050 2350
-F 0 "#PWR0110" H 4050 2200 50  0001 C CNN
-F 1 "+5V" H 4000 2525 50  0000 C CNN
-F 2 "" H 4050 2350 50  0001 C CNN
-F 3 "" H 4050 2350 50  0001 C CNN
-	1    4050 2350
-	1    0    0    -1
-$EndComp
-$Comp
-L power:+3.3V #PWR0117
-U 1 1 5FB43EC1
-P 4650 2350
-F 0 "#PWR0117" H 4650 2200 50  0001 C CNN
-F 1 "+3.3V" H 4700 2525 50  0000 C CNN
-F 2 "" H 4650 2350 50  0001 C CNN
-F 3 "" H 4650 2350 50  0001 C CNN
-	1    4650 2350
-	1    0    0    -1
-$EndComp
-$Comp
-L Jumper:SolderJumper_3_Open JP3
-U 1 1 5FDA0480
-P 4350 2450
-F 0 "JP3" V 4350 2518 50  0000 L CNN
-F 1 "SolderJumper_3_Open" V 4395 2518 50  0001 L CNN
-F 2 "Connectors:GS3" H 4350 2450 50  0001 C CNN
-F 3 "~" H 4350 2450 50  0001 C CNN
-	1    4350 2450
-	1    0    0    -1
-$EndComp
-Wire Wire Line
-	4350 2600 4350 2775
-Connection ~ 4350 2775
-Wire Wire Line
-	4350 2775 4350 3275
-Wire Wire Line
-	4650 2450 4550 2450
-Wire Wire Line
-	4650 2350 4650 2450
-Wire Wire Line
-	4150 2450 4050 2450
-Wire Wire Line
-	4050 2450 4050 2350
 $EndSCHEMATC
