File: kicad/stima_v4/Stima V4 Slave Rev1_1_Ki/Stima V4 Slave R1_1.kicad_pcb (KiCad board)
At the start: 4 copper layers, 130 x 74.7 mm, 290 parts, among them J1 Pico Blade 8p 53398-0871, J10 8P, J11 VIAS1, J12 2P, J2 6P, J3 3P, J4 3P, J5 5P, J6 Pico-Clasp, J7 4P, J8 6P, J9 4P, SW1 B3F xx, U1 STM32L452RCT6, U10 TRSF3232EIDR, U11 IIS328DQ, U12 OPA2735, U13 OPA2735, U14 TXU0204, U15 AP22653, U16 BTS72004, U17 ST732, U18 AP22653, U19 MAX20077ATCA/VY+, U2 CAT24C64, U20 ST732, U3 AT25SF, U4 TJA1443ATK, U5 PCA9616, U6 PCA9517D, U7 ST732, U8 AP22653, U9 AP22653, X1 32.768KHz

Commit message: Update KiCad Stima V4
Add KiCad Stima V4 project
Parts:
- removed +12V, +3V3S, +5V, GND: TestPoint, ARGO Passive Component.IntLib:TP
- removed the ? at (161.7, 110.6)
- removed CS1: Circuito Stampato, ARGO.PcbLib:CS
- added +12V1: TestPoint, Library_Slave_impronte:TP, F.Cu at (142.0, 92.6)
- added +3V3S1: TestPoint, Library_Slave_impronte:TP, F.Cu at (175.3, 124.6)
- added +5V1: TestPoint, Library_Slave_impronte:TP, F.Cu at (159.8, 91.5)
- added ?: , Library_Slave_impronte:_Altium_Library_ARGO_ARGO PcbLib-Trad1.PcbLib_CapELSUPERCAP FT0H104ZF, B.Cu at (161.7, 110.5)
- added GND1: TestPoint, Library_Slave_impronte:TP, F.Cu at (159.8, 96.6)
- +3V3: footprint ARGO Passive Component.IntLib:TP -> Library_Slave_impronte:TP
- A1, A2, A3, A4: footprint ARGO PcbLib-Trad1.PcbLib:ViteDado4 -> Library_Slave_impronte:ViteDado4
- A5: footprint ARGO Passive Component.IntLib:ViteDado4 -> Library_Slave_impronte:ViteDado4
- A6: footprint ARGO Passive Component.IntLib:ViteDado3 -> Library_Slave_impronte:ViteDado4
- C1, C10, C11, C8, C9: value 4.7u -> 4.7uF; footprint ARGO Passive Component.IntLib:0603 -> Library_Slave_impronte:0603
- C12, C15, C3: value 100n -> 100nF; footprint ARGO Passive Component.IntLib:0603 -> Library_Slave_impronte:0805
- C13, C14, C28, C29, C30, C33, C34, C35, C38, C49, C55, C57, C60, C62, C63, C66, C67, C70, C71, C72, C73, C74, C76, C77, C80, C83, C85, C87, C88, C89, C90, FIL2, FIL3, FIL4, FIL5, FIL6, FIL7, R1, R10, R13, R14, R15, R16, R17, R18, R19, R2, R20, R22, R23, R24, R25, R26, R27, R28, R3, R30, R31, R32, R33, R34, R35, R36, R37, R38, R4, R40, R41, R42, R43, R44, R45, R46, R47, R48, R49, R5, R50, R51, R52, R53, R54, R55, R56, R57, R58, R59, R6, R60, R61, R62, R63, R64, R65, R66, R67, R68, R69, R7, R70, R72, R76, R77, R78, R79, R8, R9: footprint ARGO Passive Component.IntLib:0603 -> Library_Slave_impronte:0603
- C16: footprint ARGO Passive Component.IntLib:10X8-10_5 -> Library_Slave_impronte:10X8-10_5
- C17, C2, C21, C22, C23, C24, C26, C27, C31, C32, C36, C37, C39, C4, C42, C43, C44, C47, C48, C5, C50, C51, C52, C53, C58, C6, C64, C65, C68, C7, C75, C78, C79, C86: value 100n -> 100nF; footprint ARGO Passive Component.IntLib:0603 -> Library_Slave_impronte:0603
- C18, C19, C20, C25, C69: value 220p -> 220pF; footprint ARGO Passive Component.IntLib:0603 -> Library_Slave_impronte:0603
- C40, C41, C45, C46: value 100p -> 100pF; footprint ARGO Passive Component.IntLib:0603 -> Library_Slave_impronte:0603
- C54, C56, C59, C61: value 470p -> 470pF; footprint ARGO Passive Component.IntLib:0603 -> Library_Slave_impronte:0603
- C81: value 100n -> 100nF; footprint ARGO Passive Component.IntLib:0805 -> Library_Slave_impronte:0805
- C82: footprint ARGO Passive Component.IntLib:1206 -> Library_Power_impronte:1206
- C84: footprint ARGO Passive Component.IntLib:0805 -> Library_Slave_impronte:0603
- D1: footprint ARGO Passive Component.IntLib:DO-214AB -> Library_Slave_impronte:DO-214AB
- DL1: footprint ARGO Passive Component.IntLib:0805-led -> Library_Slave_impronte:0805-led
- DZ1, DZ2: footprint ARGO Passive Component.IntLib:QFN-3L-DFN1110 -> Library_Slave_impronte:QFN-3L-DFN1110
- DZ10, DZ11, DZ12, DZ13, DZ15, DZ16, DZ17, DZ18, DZ19, DZ5, DZ6, DZ7, DZ8, DZ9: footprint ARGO Passive Component.IntLib:SOD 523(SC-79) -> Library_Slave_impronte:SOD 523(SC-79)
- DZ14: value PESD5Z12 -> PESD5Z12,115; footprint ARGO Passive Component.IntLib:SOD 523(SC-79) -> Library_Slave_impronte:SOD 523(SC-79)
- DZ3: footprint ARGO.PcbLib:SMA -> Library_Slave_impronte:SMA
- F1: value MF- -> MF-NSMF150; footprint ARGO Passive Component.IntLib:1206 -> Library_Slave_impronte:1206
- FIL1: value BLM18BD -> BLM18BD102SN1D; footprint ARGO Passive Component.IntLib:0603 -> Library_Slave_impronte:0603
- FIL11, FIL12, FIL13, FIL14: footprint ARGO Passive Component.IntLib:NFM18PS -> Library_Slave_impronte:NFM18PS
- FIL15: footprint ARGO.PcbLib:NFE61PT-2606 -> Library_Slave_impronte:NFE61PT-2606
- J1: footprint ARGO Passive Component.IntLib:MOLEX8P1_25SMD -> Library_Slave_impronte:MOLEX8P1_25SMD
- J10: footprint ARGO Passive Component.IntLib:CONN_8P-P381 -> Library_Slave_impronte:CONN_8P-P381
- J11: footprint ARGO PcbLib-Trad1.PcbLib:VIAS0_8 -> Library_Slave_impronte:VIAS0_8
- J12: footprint ARGO Passive Component.IntLib:CONN_2P-P381 -> Library_Slave_impronte:CONN_2P-P381
- J2, J8: footprint ARGO Passive Component.IntLib:CONN_6P-P381 -> Library_Slave_impronte:CONN_6P-P381
- J3, J4: footprint ARGO Passive Component.IntLib:CONN_3P-P381 -> Library_Slave_impronte:CONN_3P-P381
- J5: footprint ARGO Passive Component.IntLib:CONN_5P-P381 -> Library_Slave_impronte:CONN_5P-P381
- J6: value Pico-Clasp -> Pico-Clasp 6p 5015680607; footprint ARGO.PcbLib:PICOCLASP6P_REV-MIO -> Library_Slave_impronte:PICOCLASP6P_REV-MIO
- J7, J9: footprint ARGO Passive Component.IntLib:CONN_4P-P381 -> Library_Slave_impronte:CONN_4P-P381
- JP1, JP6, JP7: footprint ARGO PcbLib-Trad1.PcbLib:STRIP3PP254 -> Library_Slave_impronte:STRIP3PP254
- JP10, JP11, JP12, JP13, JP14, JP15, JP16, JP17, JP18, JP19, JP2, JP20, JP21, JP22, JP23, JP24, JP25, JP26, JP27, JP28, JP29, JP3, JP30, JP31, JP32, JP33, JP34, JP35, JP4, JP5, JP8, JP9: footprint ARGO Passive Component.IntLib:STRIP2P -> Library_Slave_impronte:STRIP2P
- L1: value ACT45B-110 -> ACT45B-110-2P-TL003; footprint ARGO Passive Component.IntLib:ACT45B TDK-MIO -> Library_Slave_impronte:ACT45B TDK-MIO
- L2: value XAL4020 -> XAL4020-222MEC; footprint ARGO.PcbLib:COIL COILCRAFT XAL4020-MIO -> Library_Slave_impronte:COIL COILCRAFT XAL4020-MIO
- L3: footprint ARGO Miscellanea.IntLib:FILTRO DLW5B -> Library_Slave_impronte:FILTRO DLW5B
- OC1, OC2, OC3: value TLP292 -> TLP292GB; footprint ARGO Miscellanea.IntLib:SO4-OPTO -> Library_Slave_impronte:SO4-OPTO
- R11, R12: value 60R4 -> MMA0204 60R4; footprint ARGO.PcbLib:MELFRESMMA0204 -> Library_Slave_impronte:MELFRESMMA0204
- R21, R29, R39, R71, R73, R74, R75: footprint ARGO Passive Component.IntLib:0805 -> Library_Slave_impronte:0805
- SW1: footprint ARGO Passive Component.IntLib:TASTO SMD 6X6 -> Library_Slave_impronte:TASTO SMD 6X6
- U1: footprint ARGO Texas.IntLib:LQFP64 -> Library_Slave_impronte:LQFP64
- U10: footprint ARGO Texas.IntLib:SO16 -> Library_Slave_impronte:SO16
- U11: footprint ARGO Miscellanea.IntLib:VQFN24 -> Library_Slave_impronte:VQFN24
- U12, U13: value OPA2735 -> OPA2735AID; footprint ARGO BurrBrown.IntLib:SO8 -> Library_Slave_impronte:SO8
- U14: value TXU0204 -> TXU0204QPWRQ1; footprint ARGO Texas.IntLib:TSSOP14 -> Library_Slave_impronte:TSSOP14
- U15, U18, U8, U9: value AP22653 -> AP22653QW6-7; footprint ARGO.PcbLib:SOT26 -> Library_Slave_impronte:SOT26
- U16: value BTS72004 -> BTS72004EPAXUMA1; footprint ARGO Miscellanea.IntLib:TSDSO-14 -> Library_Slave_impronte:TSDSO-14
- U17, U20: value ST732 -> ST732M33R; footprint ARGO Miscellanea.IntLib:SOT23_5 -> Library_Slave_impronte:SOT23_5
- U19: footprint ARGO.PcbLib:TDFN 12L -> Library_Slave_impronte:TDFN 12L
- U2: value CAT24C64 -> CAT24C64WI; footprint ARGO Miscellanea.IntLib:SO8 -> Library_Slave_impronte:SO8
- U3: value AT25SF -> AT25SF161SSHD; footprint ARGO Texas.IntLib:SO8 -> Library_Slave_impronte:SO8
- U4: footprint ARGO Miscellanea.IntLib:HVSON14 -> Library_Slave_impronte:HVSON14
- U5: value PCA9616 -> NM PCA9616PW; footprint ARGO Miscellanea.IntLib:TSSOP16 -> Library_Slave_impronte:TSSOP16
- U6: value PCA9517D -> PCA9517D (TCA9517D); footprint ARGO Miscellanea.IntLib:SO8 -> Library_Slave_impronte:SO8
- U7: value ST732 -> ST732M50R; footprint ARGO Miscellanea.IntLib:SOT23_5 -> Library_Slave_impronte:SOT23_5
- X1: footprint ARGO.PcbLib:CRYST_ECS -> Library_Slave_impronte:CRYST_ECS
- moved R79 0.86 mm to (153.5, 129.8)
- moved R77 0.81 mm to (122.9, 94.5)
- moved R78 0.61 mm to (121.7, 90.3)
- moved C3 0.48 mm to (141.0, 122.7)
Connections:
- net -RESET renamed /Stima V4 Slave_Cpu R1_1/-RESET
- net AIN1 renamed /Stima V4 Slave_Input R1_1/AIN1
- net AIN2 renamed /Stima V4 Slave_Input R1_1/AIN2
- net AIN3 renamed /Stima V4 Slave_Input R1_1/AIN3
- net AIN4 renamed /Stima V4 Slave_Input R1_1/AIN4
- net CANH renamed /Stima V4 Slave_I2C&Can R1_1/CANH
- net CANL renamed /Stima V4 Slave_I2C&Can R1_1/CANL
- net DIN0 renamed /Stima V4 Slave_Input R1_1/DIN0
- net DIN1 renamed /Stima V4 Slave_Input R1_1/DIN1
- net DIN2 renamed /Stima V4 Slave_Input R1_1/DIN2
- net F_-CS renamed /Stima V4 Slave_Cpu R1_1/F_-CS
- net F_I/O0 renamed /Stima V4 Slave_Cpu R1_1/F_I/O0
- net F_I/O1 renamed /Stima V4 Slave_Cpu R1_1/F_I/O1
- net F_I/O2 renamed /Stima V4 Slave_Cpu R1_1/F_I/O2
- net F_I/O3 renamed /Stima V4 Slave_Cpu R1_1/F_I/O3
- net F_SCK renamed /Stima V4 Slave_Cpu R1_1/F_SCK
- net NetC13_1 renamed Net-(U1-PC14/OSC32_IN)
- net NetC14_1 renamed Net-(U1-PC15/OSC32_OUT)
- net NetC15_1 renamed Net-(U1-VBAT)
- net NetC16_1 renamed Net-(C16-Pad1)
- net NetC19_2 renamed Net-(U4-CANH)
- net NetC1_1 renamed Net-(U1-VDDA/VREF+)
- net NetC20_2 renamed Net-(U4-CANL)
- net NetC21_2 renamed Net-(C21-Pad2)
- net NetC27_1 renamed Net-(U6-VCCB)
- net NetC34_1 renamed Net-(U7-VOUT)
- net NetC39_1 renamed Net-(U10-C1-)
- net NetC39_2 renamed Net-(U10-C1+)
- net NetC40_2 renamed Net-(C40-Pad2)
- net NetC41_2 renamed Net-(DZ6-K)
- net NetC42_2 renamed Net-(U10-V+)
- net NetC43_1 renamed Net-(U10-C2-)
- net NetC43_2 renamed Net-(U10-C2+)
- net NetC44_2 renamed Net-(U10-V-)
- net NetC45_2 renamed Net-(C45-Pad2)
- net NetC46_2 renamed Net-(DZ7-K)
- net NetC50_1 renamed Net-(U14-VCCB)
- net NetC54_1 renamed ADC1_IN1
- net NetC55_1 renamed Net-(DZ9-K)
- net NetC56_1 renamed ADC1_IN2
- net NetC57_1 renamed Net-(DZ11-K)
- net NetC59_1 renamed ADC1_IN3
- net NetC60_1 renamed Net-(DZ13-K)
- net NetC61_1 renamed ADC1_IN4
- net NetC62_1 renamed Net-(DZ15-K)
- net NetC67_2 renamed Net-(U16-GND)
- net NetC69_1 renamed IS
- net NetC79_1 renamed Net-(FIL15-I)
- net NetC81_1 renamed Net-(U19-BST)
- net NetC81_2 renamed Net-(U19-LX)
- net NetC84_2 renamed Net-(U19-BIAS)
- net NetD1_1 renamed Net-(D1-K)
- net NetD1_2 renamed Net-(D1-A)
- net NetDL1_1 renamed Net-(DL1-K)
- net NetDL1_2 renamed Net-(DL1-A)
- net NetDZ16_1 renamed Net-(DZ16-K)
- net NetF1_2 renamed Net-(F1-Pad2)
- net NetFIL11_2 renamed Net-(FIL11-O)
- net NetFIL12_2 renamed Net-(FIL12-O)
- net NetFIL13_2 renamed Net-(FIL13-O)
- net NetFIL14_2 renamed Net-(FIL14-O)
- net NetFIL4_1 renamed Net-(U10-DO1)
- net NetFIL4_2 renamed Net-(FIL4-Pad2)
- net NetFIL5_1 renamed Net-(U10-DO2)
- net NetFIL5_2 renamed Net-(FIL5-Pad2)
- net NetFIL6_1 renamed Net-(U10-RIN1)
- net NetFIL6_2 renamed Net-(FIL6-Pad2)
- net NetFIL7_1 renamed Net-(U10-RIN2)
- net NetFIL7_2 renamed Net-(FIL7-Pad2)
- net NetJ1_2 renamed Net-(J1-Pad2)
- net NetJ1_6 renamed Net-(J1-Pad6)
- net NetJ2_2 renamed Net-(U5-DSDAM)
- net NetJ2_4 renamed Net-(U5-DSCLM)
- net NetJ6_2 renamed Net-(U14-B2Y)
- net NetJ6_3 renamed Net-(U14-B3)
- net NetJ6_4 renamed Net-(U14-B1Y)
- net NetJP10_2 renamed Net-(JP10-Pad2)
- net NetJP11_2 renamed Net-(JP11-Pad2)
- net NetJP12_2 renamed Net-(JP12-Pad2)
- net NetJP13_2 renamed Net-(JP13-Pad2)
- net NetJP14_2 renamed Net-(JP14-Pad2)
- net NetJP15_2 renamed Net-(JP15-Pad2)
- net NetJP16_2 renamed Net-(JP16-Pad2)
- net NetJP17_2 renamed Net-(JP17-Pad2)
- net NetJP18_2 renamed Net-(JP18-Pad2)
- net NetJP19_2 renamed Net-(JP19-Pad2)
- net NetJP20_2 renamed Net-(JP20-Pad2)
- net NetJP21_2 renamed Net-(JP21-Pad2)
- net NetJP22_2 renamed Net-(JP22-Pad2)
- net NetJP23_2 renamed Net-(JP23-Pad2)
- net NetJP24_2 renamed Net-(JP24-Pad2)
- net NetJP25_2 renamed Net-(JP25-Pad2)
- net NetJP26_2 renamed Net-(JP26-Pad2)
- net NetJP27_2 renamed Net-(JP27-Pad2)
- net NetJP28_2 renamed Net-(JP28-Pad2)
- net NetJP29_2 renamed Net-(JP29-Pad2)
- net NetJP2_1 renamed Net-(U1-PH3/BOOT0)
- net NetJP30_2 renamed Net-(JP30-Pad2)
- net NetJP31_2 renamed Net-(JP31-Pad2)
- net NetJP32_2 renamed Net-(JP32-Pad2)
- net NetJP33_1 renamed Net-(JP33-Pad1)
- net NetJP33_2 renamed Net-(JP33-Pad2)
- net NetJP34_1 renamed Net-(JP34-Pad1)
- net NetJP34_2 renamed Net-(JP34-Pad2)
- net NetJP35_1 renamed Net-(JP35-Pad1)
- net NetJP35_2 renamed Net-(JP35-Pad2)
- net NetJP3_2 renamed Net-(JP3-Pad2)
- net NetJP4_2 renamed Net-(JP4-Pad2)
- net NetJP5_1 renamed Net-(JP5-Pad1)
- net NetJP8_2 renamed Net-(JP8-Pad2)
- net NetJP9_2 renamed Net-(JP9-Pad2)
- net NetR13_1 renamed I2C2_SCL
- net NetR14_1 renamed I2C2_SDA
- net NetR15_1 renamed Net-(U8-ILIM)
- net NetR16_1 renamed Net-(U9-ILIM)
- net NetR20_1 renamed Net-(U12A-IN-)
- net NetR32_1 renamed Net-(U12B-IN-)
- net NetR43_1 renamed Net-(U13A-IN-)
- net NetR50_1 renamed Net-(U13B-IN-)
- net NetR57_1 renamed Net-(U15-ILIM)
- net NetR58_1 renamed DEN
- net NetR58_2 renamed Net-(U16-DEN)
- net NetR60_1 renamed DSEL0
- net NetR60_2 renamed Net-(U16-DSEL0)
- net NetR61_1 renamed Net-(U16-IS)
- net NetR63_1 renamed DSEL1
- net NetR63_2 renamed Net-(U16-DSEL1)
- net NetR65_1 renamed PW0
- net NetR65_2 renamed Net-(U16-IN0)
- net NetR66_1 renamed PW1
- net NetR66_2 renamed Net-(U16-IN1)
- net NetR67_1 renamed PW2
- net NetR67_2 renamed Net-(U16-IN2)
- net NetR68_1 renamed PW3
- net NetR68_2 renamed Net-(U16-IN3)
- net NetR69_2 renamed FAULT
- net NetR6_2 renamed Net-(U2-WP)
- net NetR70_1 renamed Net-(U18-ILIM)
- net NetR72_1 renamed Net-(U19-SPS)
- net NetR76_2 renamed Net-(U5-VDDA_SEL)
- net NetR79_1 renamed Net-(U1-PH0/OSC_IN)
- net NetU1_14 renamed 232_CTS
- net NetU1_15 renamed 232_RTS
- net NetU1_16 renamed 232_TX
- net NetU1_21 renamed SPI_SCK
- net NetU1_33 renamed CAN1_RX
- net NetU1_34 renamed CAN1_TX
- net NetU1_36 renamed STB_CAN
- net NetU1_44 renamed SPI_MISO
- net NetU1_45 renamed SPI_MOSI
- net NetU1_50 renamed 232_RX
- net NetU1_52 renamed I2C2_EN
- net NetU1_53 renamed EN_CAN
- net NetU1_54 renamed EN_SPLY
- net NetU1_57 renamed EN_5VS
- net NetU1_62 renamed EN_5VA
- net SCL renamed /Stima V4 Slave_I2C&Can R1_1/SCL
- net SDA renamed /Stima V4 Slave_I2C&Can R1_1/SDA
- net SWCLK renamed /Stima V4 Slave_Cpu R1_1/SWCLK
- net SWDIO renamed /Stima V4 Slave_Cpu R1_1/SWDIO
- net SWO renamed /Stima V4 Slave_Cpu R1_1/SWO
- A1 pad 1: (no net) -> unconnected-(A1-A-Pad1)
- A2 pad 1: (no net) -> unconnected-(A2-A-Pad1)
- A3 pad 1: (no net) -> unconnected-(A3-A-Pad1)
- A4 pad 1: (no net) -> unconnected-(A4-A-Pad1)
- A5 pad 1: (no net) -> unconnected-(A5-A-Pad1)
- A6 pad 1: (no net) -> unconnected-(A6-A-Pad1)
- JP1 pad 2: RXD -> /Stima V4 Slave_Cpu R1_1/RXD1
- JP1 pad 3: NetJP1_3 -> RXD
- R18 pad 1: NetJP1_3 -> RXD
- SW1 pad 4: (no net) -> unconnected-(SW1-Pad4)
- U1 pad 2: (no net) -> unconnected-(U1-PC13-Pad2)
- U1 pad 43: RXD -> /Stima V4 Slave_Cpu R1_1/RXD1
- U1 pad 6: (no net) -> unconnected-(U1-PH1/OSC_OUT-Pad6)
- U11 pad 1: (no net) -> unconnected-(U11-NC-Pad1)
- U11 pad 12: (no net) -> unconnected-(U11-CS-Pad12)
- U11 pad 15: (no net) -> unconnected-(U11-SA0/SDO-Pad15)
- U11 pad 17: (no net) -> unconnected-(U11-NC-Pad17)
- U11 pad 18: (no net) -> unconnected-(U11-NC-Pad18)
- U11 pad 19: (no net) -> unconnected-(U11-NC-Pad19)
- U11 pad 2: (no net) -> unconnected-(U11-NC-Pad2)
- U11 pad 20: (no net) -> unconnected-(U11-NC-Pad20)
- U11 pad 21: (no net) -> unconnected-(U11-NC-Pad21)
- U11 pad 22: (no net) -> unconnected-(U11-NC-Pad22)
- U11 pad 23: (no net) -> unconnected-(U11-NC-Pad23)
- U11 pad 24: (no net) -> unconnected-(U11-NC-Pad24)
- U11 pad 3: (no net) -> unconnected-(U11-INT_2-Pad3)
- U11 pad 7: (no net) -> unconnected-(U11-INT_1-Pad7)
- U14 pad 5: (no net) -> unconnected-(U14-A4Y-Pad5)
- U14 pad 6: (no net) -> unconnected-(U14-NC-Pad6)
- U14 pad 9: (no net) -> unconnected-(U14-NC-Pad9)
- U15 pad 4: (no net) -> unconnected-(U15-\~{FLT}-Pad4)
- U16 pad 3: (no net) -> unconnected-(U16-NC-Pad3)
- U17 pad 4: (no net) -> unconnected-(U17-NC-Pad4)
- U17 pad 5: (no net) -> unconnected-(U17-NC-Pad5)
- U20 pad 4: (no net) -> unconnected-(U20-NC-Pad4)
- U20 pad 5: (no net) -> unconnected-(U20-NC-Pad5)
- U4 pad 11: (no net) -> unconnected-(U4-NC-Pad11)
- U4 pad 7: (no net) -> unconnected-(U4-INH-Pad7)
- U4 pad 8: (no net) -> unconnected-(U4-ERR_N-Pad8)
- U4 pad 9: (no net) -> unconnected-(U4-WAKE-Pad9)
- U5 pad 10: (no net) -> unconnected-(U5-DINTP-Pad10)
- U5 pad 11: (no net) -> unconnected-(U5-DINTM-Pad11)
- U5 pad 5: (no net) -> unconnected-(U5-\~{PIDET}-Pad5)
- U5 pad 6: (no net) -> unconnected-(U5-\~{READY}-Pad6)
- U5 pad 7: (no net) -> unconnected-(U5-INT-Pad7)
- U7 pad 4: (no net) -> unconnected-(U7-NC-Pad4)
- U7 pad 5: (no net) -> unconnected-(U7-NC-Pad5)
- U8 pad 4: (no net) -> unconnected-(U8-\~{FLT}-Pad4)
- U9 pad 4: (no net) -> unconnected-(U9-\~{FLT}-Pad4)
Routing:
- net /Stima V4 Slave_Cpu R1_1/RXD1: track 0.00 -> 19.3 mm, vias 0 -> 1
- net RXD: track 19.3 -> 8.41 mm
- net NetJP1_3: track 8.41 -> 0.00 mm, vias 1 -> 0
Other:
- board text added: ".Pcb_File_Name_No_Path"
- board text added: ".Print_Date"
- board text added: ".Print_Time"
- board text added: "1"
- board text added: "1.1"
- board text added: "1:1"
- board text added: "2"
- board text added: "4"
- board text added: "A"
- board text added: "B"
- board text added: "C"
- board text added: "D"
- board text added: "DATE:"
- board text added: "DWG NO:"
- board text added: "FILE NAME:"
- board text added: "G. Cocchi"
- board text added: "PART NO.:"
- board text added: "PCB DESIGNER:"
- board text added: "REV:"
- board text added: "SCALE:"
- board text added: "Stima V4-Slave"
- board text added: "TITLE:"
- board text added: "Time:"
