File: kicad/stima_v4/Stima V4 Slave Rev1_1_Ki/Stima V4 Slave_Cpu R1_1.kicad_sch (KiCad schematic)
At the start: 38 parts, among them J1 Pico Blade 8p 53398-0871, SW1 B3F xx, U1 STM32L452RCT6, U2 CAT24C64WI, U3 AT25SF161SSHD, X1 32.768KHz

Commit message: Update KiCad Stima V4
Add KiCad Stima V4 project
Parts:
- C1, C10, C11, C13, C14, C17, C2, C4, C5, C6, C7, C8, C9, FIL1, R1, R10, R2, R3, R4, R5, R6, R7, R79, R8, R9: footprint 0603 -> Library_Slave_impronte:0603
- C12, C15, C3: footprint 0603 -> Library_Slave_impronte:0805
- C16: footprint 10X8-10_5 -> Library_Slave_impronte:10X8-10_5
- J1: footprint MOLEX8P1_25SMD -> Library_Slave_impronte:MOLEX8P1_25SMD
- JP1: footprint STRIP3PP254 -> Library_Slave_impronte:STRIP3PP254
- JP2, JP3: footprint STRIP2P -> Library_Slave_impronte:STRIP2P
- SW1: footprint TASTO SMD 6X6 -> Library_Slave_impronte:TASTO SMD 6X6
- U1: footprint LQFP64 -> Library_Slave_impronte:LQFP64
- U2, U3: footprint SO8 -> Library_Slave_impronte:SO8
- X1: footprint CRYST_ECS -> Library_Slave_impronte:CRYST_ECS
Connections:
- net RXD: no longer JP1.2, U1.43 (PA10)
- new net RXD1: JP1.2, U1.43 (PA10)
- no-connect marks 0 -> 2
Other:
- note added: "${##}"
- note added: "${CURRENT_DATE}"
- note added: "${DOCUMENTNUMBER}"
- note added: "${FILENAME}"
- note added: "${TITLE}"
- note added: "1.1"
- note added: "A4"
- note added: "Date:"
- note added: "Number:"
- note added: "Revision:"
- note added: "Sheet"
- note added: "Size:"
- note added: "Title"
- note added: "of"
- note removed: "6"
- moved on the sheet: C1, C10, C11, C12, C13, C14, C15, C16, C17, C2, C3, C4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
