File: kicad/stima_v4/Stima V4 Slave Rev1_1_Ki/Stima V4 Slave_Input R1_1.kicad_sch (KiCad schematic)
At the start: 103 parts, among them J7 4P, J8 6P, U12 OPA2735AID, U13 OPA2735AID, U15 AP22653QW6-7

Commit message: Update KiCad Stima V4
Add KiCad Stima V4 project
Parts:
- C53, C54, C55, C56, C57, C58, C59, C60, C61, C62, C63, C64, C65, C66, R19, R20, R22, R23, R24, R25, R26, R27, R28, R30, R31, R32, R33, R34, R35, R36, R37, R38, R40, R41, R42, R43, R44, R45, R46, R47, R48, R49, R50, R51, R52, R53, R54, R55, R56, R57: footprint 0603 -> Library_Slave_impronte:0603
- DZ10, DZ11, DZ12, DZ13, DZ14, DZ15, DZ8, DZ9: footprint SOD 523(SC-79) -> Library_Slave_impronte:SOD 523(SC-79)
- FIL11, FIL12, FIL13, FIL14: footprint NFM18PS -> Library_Slave_impronte:NFM18PS
- J7: footprint CONN_4P-P381 -> Library_Slave_impronte:CONN_4P-P381
- J8: footprint CONN_6P-P381 -> Library_Slave_impronte:CONN_6P-P381
- JP10, JP11, JP12, JP13, JP14, JP15, JP16, JP17, JP18, JP19, JP20, JP21, JP22, JP23, JP24, JP25, JP26, JP27, JP28, JP29, JP30, JP31, JP33, JP34, JP35, JP8, JP9: footprint STRIP2P -> Library_Slave_impronte:STRIP2P
- OC1, OC2, OC3: footprint SO4-OPTO -> Library_Slave_impronte:SO4-OPTO
- R21, R29, R39, R73, R74, R75: footprint 0805 -> Library_Slave_impronte:0805
- U12, U13: footprint SO8 -> Library_Slave_impronte:SO8
- U15: footprint SOT26 -> Library_Slave_impronte:SOT26
Connections:
- no-connect marks 0 -> 1
Other:
- note added: "${##}"
- note added: "${CURRENT_DATE}"
- note added: "${DOCUMENTNUMBER}"
- note added: "${FILENAME}"
- note added: "${TITLE}"
- note added: "1.1"
- note added: "A4"
- note added: "Customer:"
- note added: "Date:"
- note added: "Number:"
- note added: "Project by:"
- note added: "Revision:"
- note added: "Sheet"
- note added: "Size:"
- note added: "Title"
- note added: "of"
- note removed: "6"
- moved on the sheet: C53, C54, C55, C56, C57, C58, C59, C60, C61, C62, C63, C64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
