File: kicad/stima_v4/Stima V4 Slave Rev1_1_Ki/Stima V4 Slave_Power R1_1.kicad_sch (KiCad schematic)
At the start: 34 parts, among them J11 VIAS1, J12 2P, U19 MAX20077ATCA/VY+, U20 ST732M33R

Commit message: Update KiCad Stima V4
Add KiCad Stima V4 project
Parts:
- removed +12V, +3V3, +5V: TestPoint, TP, symbol Stima V4 Slave Rev1_1-altium-import:root_1_TestPoint
- removed GND: TestPoint, TP, symbol Stima V4 Slave Rev1_1-altium-import:root_3_TestPoint
- added +12V1, +3V3, +5V1, GND1: TestPoint, Library_Slave_impronte:TP, symbol Connector:TestPoint
- A1, A2, A3, A4, A5: footprint ViteDado4 -> Library_Slave_impronte:ViteDado4
- A6: footprint ViteDado3 -> Library_Slave_impronte:ViteDado4
- C81, R71: footprint 0805 -> Library_Slave_impronte:0805
- C82: footprint 1206 -> Library_Power_impronte:1206
- C83, C85, C86, C87, C88, C89, C90, R72: footprint 0603 -> Library_Slave_impronte:0603
- C84: footprint 0805 -> Library_Slave_impronte:0603
- D1: footprint DO-214AB -> Library_Slave_impronte:DO-214AB
- DL1: footprint 0805-led -> Library_Slave_impronte:0805-led
- DZ19: footprint SOD 523(SC-79) -> Library_Slave_impronte:SOD 523(SC-79)
- DZ3: footprint SMA -> Library_Slave_impronte:SMA
- F1: footprint 1206 -> Library_Slave_impronte:1206
- J11: footprint VIAS0_8 -> Library_Slave_impronte:VIAS0_8
- J12: footprint CONN_2P-P381 -> Library_Slave_impronte:CONN_2P-P381
- JP32: footprint STRIP2P -> Library_Slave_impronte:STRIP2P; PACKAGE REFERENCE (none) -> PTH
- L2: footprint COIL COILCRAFT XAL4020-MIO -> Library_Slave_impronte:COIL COILCRAFT XAL4020-MIO
- L3: footprint FILTRO DLW5B -> Library_Slave_impronte:FILTRO DLW5B
- U19: footprint TDFN 12L -> Library_Slave_impronte:TDFN 12L
- U20: footprint SOT23_5 -> Library_Slave_impronte:SOT23_5
Connections:
- net +12V: now also +12V1.1
- net +3V3: now also +3V3.1
- net +5V: now also +5V1.1
- net GND: now also GND1.1
- no-connect marks 0 -> 6
Other:
- note added: "${##}"
- note added: "${CURRENT_DATE}"
- note added: "${DOCUMENTNUMBER}"
- note added: "${FILENAME}"
- note added: "${TITLE}"
- note added: "1.1"
- note added: "A4"
- note added: "Customer:"
- note added: "Date:"
- note added: "Number:"
- note added: "Project by:"
- note added: "Revision:"
- note added: "Sheet"
- note added: "Size:"
- note added: "Title"
- note added: "of"
- note removed: "6"
