File: kicad/stima_v4/Stima V4 Slave Rev1_1_Ki/Stima V4 Slave_PowerSensor R1_1.kicad_sch (KiCad schematic)
At the start: 38 parts, among them J10 8P, J9 4P, U16 BTS72004EPAXUMA1, U17 ST732M33R, U18 AP22653QW6-7

Commit message: Update KiCad Stima V4
Add KiCad Stima V4 project
Parts:
- removed CS1: Circuito Stampato, CS, symbol Stima V4 Slave Rev1_1-altium-import:root_0_Dummy
- +3V3S: footprint TP -> Library_Slave_impronte:TP
- C67, C68, C69, C70, C71, C72, C73, C74, C75, C76, C77, C78, C79, C80, R58, R59, R60, R61, R62, R63, R64, R65, R66, R67, R68, R69, R70: footprint 0603 -> Library_Slave_impronte:0603
- DZ16, DZ17, DZ18: footprint SOD 523(SC-79) -> Library_Slave_impronte:SOD 523(SC-79)
- FIL15: footprint NFE61PT-2606 -> Library_Slave_impronte:NFE61PT-2606
- J10: footprint CONN_8P-P381 -> Library_Slave_impronte:CONN_8P-P381
- J9: footprint CONN_4P-P381 -> Library_Slave_impronte:CONN_4P-P381
- U16: footprint TSDSO-14 -> Library_Slave_impronte:TSDSO-14
- U17: footprint SOT23_5 -> Library_Slave_impronte:SOT23_5
- U18: footprint SOT26 -> Library_Slave_impronte:SOT26
Other:
- note added: "${##}"
- note added: "${CURRENT_DATE}"
- note added: "${DOCUMENTNUMBER}"
- note added: "${FILENAME}"
- note added: "${TITLE}"
- note added: "1.1"
- note added: "A4"
- note added: "Customer:"
- note added: "Date:"
- note added: "Number:"
- note added: "Project by:"
- note added: "Revision:"
- note added: "Sheet"
- note added: "Size:"
- note added: "Title"
- note added: "of"
- note removed: "6"
- moved on the sheet: +3V3S, C67, C68, C69, C70, C71, C72, C73, C74, C75, C76, C77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
