File: kicad/stima_v4/Stima V4 Slave Rev1_1_Ki/Stima V4 Slave_RS232-SPI&Accelerometer R1_1.kicad_sch (KiCad schematic)
At the start: 31 parts, among them J4 3P, J5 5P, J6 Pico-Clasp 6p 5015680607, U10 TRSF3232EIDR, U11 IIS328DQ, U14 TXU0204QPWRQ1

Commit message: Update KiCad Stima V4
Add KiCad Stima V4 project
Parts:
- C39, C40, C41, C42, C43, C44, C45, C46, C47, C48, C49, C50, C51, C52, FIL2, FIL3, FIL4, FIL5, FIL6, FIL7, R17, R18: footprint 0603 -> Library_Slave_impronte:0603
- DZ6, DZ7: footprint SOD 523(SC-79) -> Library_Slave_impronte:SOD 523(SC-79)
- J4: footprint CONN_3P-P381 -> Library_Slave_impronte:CONN_3P-P381
- J5: footprint CONN_5P-P381 -> Library_Slave_impronte:CONN_5P-P381
- J6: footprint PICOCLASP6P_REV-MIO -> Library_Slave_impronte:PICOCLASP6P_REV-MIO
- JP7: footprint STRIP3PP254 -> Library_Slave_impronte:STRIP3PP254
- U10: footprint SO16 -> Library_Slave_impronte:SO16
- U11: footprint VQFN24 -> Library_Slave_impronte:VQFN24
- U14: footprint TSSOP14 -> Library_Slave_impronte:TSSOP14
Connections:
- no-connect marks 0 -> 5
Other:
- note added: "${##}"
- note added: "${CURRENT_DATE}"
- note added: "${DOCUMENTNUMBER}"
- note added: "${FILENAME}"
- note added: "${TITLE}"
- note added: "1.1"
- note added: "A4"
- note added: "Customer:"
- note added: "Date:"
- note added: "Number:"
- note added: "Project by:"
- note added: "Revision:"
- note added: "Sheet"
- note added: "Size:"
- note added: "Title"
- note added: "of"
- note removed: "6"
- moved on the sheet: C39, C40, C41, C42, C43, C44, C45, C46, C47, C48, C49, C50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
